File: electrical/ECU/kicad_ECU/test_shield.sch (KiCad schematic (older format))
At the start: 5 parts

Commit message: fixed some naming errors and initial round of double checking
Parts:
- removed P? (x2): CONN_01X04, symbol CONN_01X04
- removed U? (x2): 10si_rect, MODULE, symbol 10si_rect
- removed U?: Mini50p16, MODULE, symbol Mini50p16
Changed lines of the file:
@@
 $Descr A4 11693 8268
 encoding utf-8
-Sheet 10 33
+Sheet 11 33
 Title ""
 Date ""
@@
 Comment4 ""
 $EndDescr
-$Comp
-L 10si_rect U?
-U 1 1 597F7E2F
-P 5550 3300
-F 0 "U?" H 5550 3200 50  0000 C CNN
-F 1 "10si_rect" H 5550 3400 50  0000 C CNN
-F 2 "MODULE" H 5550 3300 50  0001 C CNN
-F 3 "DOCUMENTATION" H 5550 3300 50  0001 C CNN
-	1    5550 3300
-	1    0    0    -1
-$EndComp
-$Comp
-L CONN_01X04 P?
-U 1 1 597E2E29
-P 1400 4800
-F 0 "P?" H 1400 5050 50  0000 C CNN
-F 1 "CONN_01X04" V 1500 4800 50  0000 C CNN
-F 2 "" H 1400 4800 50  0000 C CNN
-F 3 "" H 1400 4800 50  0000 C CNN
-	1    1400 4800
-	-1   0    0    1
-$EndComp
-$Comp
-L CONN_01X04 P?
-U 1 1 597E2E30
-P 1450 3250
-F 0 "P?" H 1450 3500 50  0000 C CNN
-F 1 "CONN_01X04" V 1550 3250 50  0000 C CNN
-F 2 "" H 1450 3250 50  0000 C CNN
-F 3 "" H 1450 3250 50  0000 C CNN
-	1    1450 3250
-	-1   0    0    1
-$EndComp
-$Comp
-L PWR_FLAG #FLG?
-U 1 1 597E2E37
-P 2200 6750
-F 0 "#FLG?" H 2200 6845 50  0001 C CNN
-F 1 "PWR_FLAG" H 2200 6930 50  0000 C CNN
-F 2 "" H 2200 6750 50  0000 C CNN
-F 3 "" H 2200 6750 50  0000 C CNN
-	1    2200 6750
-	1    0    0    1
-$EndComp
-$Comp
-L 10si_rect U?
-U 1 1 597E2E3D
-P 1400 6650
-F 0 "U?" H 1400 6550 50  0000 C CNN
-F 1 "10si_rect" H 1400 6750 50  0000 C CNN
-F 2 "MODULE" H 1400 6650 50  0001 C CNN
-F 3 "DOCUMENTATION" H 1400 6650 50  0001 C CNN
-	1    1400 6650
-	-1   0    0    1
-$EndComp
-Text Label 2900 6650 2    60   ~ 0
-12v
-$Comp
-L PWR_FLAG #FLG?
-U 1 1 597E2E45
-P 2700 6650
-F 0 "#FLG?" H 2700 6725 50  0001 C CNN
-F 1 "PWR_FLAG" H 2700 6800 50  0000 C CNN
-F 2 "" H 2700 6650 50  0001 C CNN
-F 3 "" H 2700 6650 50  0001 C CNN
-	1    2700 6650
-	-1   0    0    1
-$EndComp
-Text Label 2450 6750 2    60   ~ 0
-BATT
-$Comp
-L Earth #PWR?
-U 1 1 597E2E4C
-P 3050 7000
-F 0 "#PWR?" H 3050 6750 50  0001 C CNN
-F 1 "Earth" H 3050 6850 50  0001 C CNN
-F 2 "" H 3050 7000 50  0001 C CNN
-F 3 "" H 3050 7000 50  0001 C CNN
-	1    3050 7000
-	1    0    0    -1
-$EndComp
-Text Label 2150 3300 2    60   ~ 0
-BOOST
-Text Label 2100 4650 2    60   ~ 0
-DF+
-Text Label 2100 4750 2    60   ~ 0
-DF-
-Text Label 2150 3100 2    60   ~ 0
-COIL1
-Text Label 2150 3400 2    60   ~ 0
-COIL2
-Text Label 2150 3200 2    60   ~ 0
-POINTS
-Text Label 2100 4850 2    60   ~ 0
-Y
-Text Label 2100 4950 2    60   ~ 0
-HC
-Wire Wire Line
-	2150 6650 2900 6650
-Wire Wire Line
-	2150 6750 2450 6750
-Wire Wire Line
-	2150 6550 3050 6550
-Wire Wire Line
-	3050 6550 3050 7000
-Wire Wire Line
-	1650 3100 2150 3100
-Wire Wire Line
-	1650 3200 2150 3200
-Wire Wire Line
-	1650 3300 2150 3300
-Wire Wire Line
-	1650 3400 2150 3400
-Wire Wire Line
-	1600 4650 2100 4650
-Wire Wire Line
-	1600 4750 2100 4750
-Wire Wire Line
-	1600 4850 2100 4850
-Wire Wire Line
-	1600 4950 2100 4950
-$Comp
-L Mini50p16 U?
-U 1 1 597E2E66
-P 2550 1400
-F 0 "U?" H 2550 1400 50  0000 C CNN
-F 1 "Mini50p16" H 2550 1600 50  0000 C CNN
-F 2 "MODULE" H 2550 1500 50  0001 C CNN
-F 3 "DOCUMENTATION" H 2550 1500 50  0001 C CNN
-	1    2550 1400
-	1    0    0    -1
-$EndComp
-Text Label 3800 1450 2    60   ~ 0
-INJ1
-Text Label 3800 1550 2    60   ~ 0
-INJ2
-Wire Wire Line
-	3800 1550 3300 1550
-Wire Wire Line
-	3300 1450 3800 1450
-Text Label 3800 1350 2    60   ~ 0
-5vOUT
-Wire Wire Line
-	3300 1350 3800 1350
-Text Label 3800 950  2    60   ~ 0
-1WIRE
-Wire Wire Line
-	3300 950  3800 950
-Text Label 3800 1850 2    60   ~ 0
-VR_lamp
-Wire Wire Line
-	3800 1850 3300 1850
-Text Label 1300 950  0    60   ~ 0
-PHASE
-Wire Wire Line
-	1300 950  1800 950
-Text Label 3800 1150 2    60   ~ 0
-O2
-Text Label 1300 1750 0    60   ~ 0
-TPS1
-Text Label 3800 1050 2    60   ~ 0
-TPS2
-Wire Wire Line
-	3300 1050 3800 1050
-Wire Wire Line
-	1300 1750 1800 1750
-Wire Wire Line
-	3300 1150 3800 1150
-Text Label 3800 1650 2    60   ~ 0
-3.3vOUT
-Wire Wire Line
-	3300 1650 3800 1650
-Wire Wire Line
-	1800 1150 1050 1150
-Wire Wire Line
-	1050 1150 1050 2100
-$Comp
-L Earth #PWR?
-U 1 1 597E2E83
-P 1050 2100
-F 0 "#PWR?" H 1050 1850 50  0001 C CNN
-F 1 "Earth" H 1050 1950 50  0001 C CNN
-F 2 "" H 1050 2100 50  0001 C CNN
-F 3 "" H 1050 2100 50  0001 C CNN
-	1    1050 2100
-	1    0    0    -1
-$EndComp
-Wire Wire Line
-	3300 1250 4050 1250
-Wire Wire Line
-	4050 1250 4050 2200
-$Comp
-L Earth #PWR?
-U 1 1 597E2E8B
-P 4050 2200
-F 0 "#PWR?" H 4050 1950 50  0001 C CNN
-F 1 "Earth" H 4050 2050 50  0001 C CNN
-F 2 "" H 4050 2200 50  0001 C CNN
-F 3 "" H 4050 2200 50  0001 C CNN
-	1    4050 2200
-	-1   0    0    -1
-$EndComp
-Text Label 1300 1050 0    60   ~ 0
-A1
-Wire Wire Line
-	1300 1050 1800 1050
-Text Label 1300 1650 0    60   ~ 0
-A2
-Wire Wire Line
-	1300 1650 1800 1650
-Text Label 1300 1850 0    60   ~ 0
-D2
-Wire Wire Line
-	1300 1850 1800 1850
-Text Label 3800 1750 2    60   ~ 0
-D1
-Wire Wire Line
-	3800 1750 3300 1750
 $EndSCHEMATC
