File: electrical/ECU/kicad_ECU/5vdc_3vdc.sch (KiCad schematic (older format))
At the start: 8 parts, among them U8 LMZ20502

Commit message: minor naming change
Parts:
- renumbered C22 to C601, C23 to C602, C24 to C603, C25 to C604, F2 to F601, R23 to R601, R24 to R602, U8 to U601
Changed lines of the file:
@@
 $EndDescr
 $Comp
-L LMZ20502 U8
+L LMZ20502 U601
 U 1 1 59718A46
 P 5350 3350
-AR Path="/597003E2/597189AE/59718A46" Ref="U8"  Part="1"
-AR Path="/5978A36B/5978B8AA/59718A46" Ref="U28"  Part="1"
-F 0 "U28" H 5350 3250 50  0000 C CNN
+AR Path="/597003E2/597189AE/59718A46" Ref="U601"  Part="1"
+AR Path="/5978A36B/5978B8AA/59718A46" Ref="U3001"  Part="1"
+F 0 "U3001" H 5350 3250 50  0000 C CNN
 F 1 "LMZ20502" H 5350 3450 50  0000 C CNN
 F 2 "MODULE" H 5350 3350 50  0001 C CNN
@@
 NoConn ~ 6100 3100
 $Comp
-L Earth #PWR032
+L Earth #PWR601
 U 1 1 59718C19
 P 4400 4600
-AR Path="/597003E2/597189AE/59718C19" Ref="#PWR032"  Part="1"
-AR Path="/5978A36B/5978B8AA/59718C19" Ref="#PWR079"  Part="1"
-F 0 "#PWR079" H 4400 4350 50  0001 C CNN
+AR Path="/597003E2/597189AE/59718C19" Ref="#PWR601"  Part="1"
+AR Path="/5978A36B/5978B8AA/59718C19" Ref="#PWR3001"  Part="1"
+F 0 "#PWR3001" H 4400 4350 50  0001 C CNN
 F 1 "Earth" H 4400 4450 50  0001 C CNN
 F 2 "" H 4400 4600 50  0001 C CNN
@@
 $EndComp
 $Comp
-L C C23
+L C C602
 U 1 1 59718C97
 P 4250 3750
-AR Path="/597003E2/597189AE/59718C97" Ref="C23"  Part="1"
-AR Path="/5978A36B/5978B8AA/59718C97" Ref="C72"  Part="1"
-F 0 "C72" H 4275 3850 50  0000 L CNN
+AR Path="/597003E2/597189AE/59718C97" Ref="C602"  Part="1"
+AR Path="/5978A36B/5978B8AA/59718C97" Ref="C3002"  Part="1"
+F 0 "C3002" H 4275 3850 50  0000 L CNN
 F 1 "10uF" H 4275 3650 50  0000 L CNN
 F 2 "" H 4288 3600 50  0001 C CNN
@@
 $EndComp
 $Comp
-L C C22
+L C C601
 U 1 1 59718CB8
 P 4000 3750
-AR Path="/597003E2/597189AE/59718CB8" Ref="C22"  Part="1"
-AR Path="/5978A36B/5978B8AA/59718CB8" Ref="C71"  Part="1"
-F 0 "C71" H 4025 3850 50  0000 L CNN
+AR Path="/597003E2/597189AE/59718CB8" Ref="C601"  Part="1"
+AR Path="/5978A36B/5978B8AA/59718CB8" Ref="C3001"  Part="1"
+F 0 "C3001" H 4025 3850 50  0000 L CNN
 F 1 "10uF" H 4025 3650 50  0000 L CNN
 F 2 "" H 4038 3600 50  0001 C CNN
@@
 $EndComp
 $Comp
-L C C24
+L C C603
 U 1 1 59718DA5
 P 7000 3350
-AR Path="/597003E2/597189AE/59718DA5" Ref="C24"  Part="1"
-AR Path="/5978A36B/5978B8AA/59718DA5" Ref="C73"  Part="1"
-F 0 "C73" H 7025 3450 50  0000 L CNN
+AR Path="/597003E2/597189AE/59718DA5" Ref="C603"  Part="1"
+AR Path="/5978A36B/5978B8AA/59718DA5" Ref="C3003"  Part="1"
+F 0 "C3003" H 7025 3450 50  0000 L CNN
 F 1 "16pF" H 7025 3250 50  0000 L CNN
 F 2 "" H 7038 3200 50  0001 C CNN
@@
 $EndComp
 $Comp
-L R R23
+L R R601
 U 1 1 59718E45
 P 6700 3050
-AR Path="/597003E2/597189AE/59718E45" Ref="R23"  Part="1"
-AR Path="/5978A36B/5978B8AA/59718E45" Ref="R99"  Part="1"
-F 0 "R99" V 6780 3050 50  0000 C CNN
+AR Path="/597003E2/597189AE/59718E45" Ref="R601"  Part="1"
+AR Path="/5978A36B/5978B8AA/59718E45" Ref="R3001"  Part="1"
+F 0 "R3001" V 6780 3050 50  0000 C CNN
 F 1 "53.2" V 6700 3050 50  0000 C CNN
 F 2 "" V 6630 3050 50  0001 C CNN
@@
 $EndComp
 $Comp
-L R R24
+L R R602
 U 1 1 59718E7C
 P 6700 3350
-AR Path="/597003E2/597189AE/59718E7C" Ref="R24"  Part="1"
-AR Path="/5978A36B/5978B8AA/59718E7C" Ref="R100"  Part="1"
-F 0 "R100" V 6780 3350 50  0000 C CNN
+AR Path="/597003E2/597189AE/59718E7C" Ref="R602"  Part="1"
+AR Path="/5978A36B/5978B8AA/59718E7C" Ref="R3002"  Part="1"
+F 0 "R3002" V 6780 3350 50  0000 C CNN
 F 1 "237" V 6700 3350 50  0000 C CNN
 F 2 "" V 6630 3350 50  0001 C CNN
@@
 $EndComp
 $Comp
-L C C25
+L C C604
 U 1 1 59718FB7
 P 7350 3050
-AR Path="/597003E2/597189AE/59718FB7" Ref="C25"  Part="1"
-AR Path="/5978A36B/5978B8AA/59718FB7" Ref="C74"  Part="1"
-F 0 "C74" H 7375 3150 50  0000 L CNN
+AR Path="/597003E2/597189AE/59718FB7" Ref="C604"  Part="1"
+AR Path="/5978A36B/5978B8AA/59718FB7" Ref="C3004"  Part="1"
+F 0 "C3004" H 7375 3150 50  0000 L CNN
 F 1 "10uF" H 7375 2950 50  0000 L CNN
 F 2 "" H 7388 2900 50  0001 C CNN
@@
 Connection ~ 7350 2900
 $Comp
-L PTC_FUSE F2
+L PTC_FUSE F601
 U 1 1 5973811D
 P 3400 3500
-AR Path="/597003E2/597189AE/5973811D" Ref="F2"  Part="1"
-AR Path="/5978A36B/5978B8AA/5973811D" Ref="F27"  Part="1"
-F 0 "F27" H 3400 3400 60  0000 C CNN
+AR Path="/597003E2/597189AE/5973811D" Ref="F601"  Part="1"
+AR Path="/5978A36B/5978B8AA/5973811D" Ref="F3001"  Part="1"
+F 0 "F3001" H 3400 3400 60  0000 C CNN
 F 1 "2A" H 3400 3300 60  0000 C CNN
 F 2 "" H 3400 3500 60  0000 C CNN
@@
 	2750 3500 3050 3500
 $Comp
-L PWR_FLAG #FLG033
+L PWR_FLAG #FLG601
 U 1 1 599195CA
 P 3800 3500
-AR Path="/597003E2/597189AE/599195CA" Ref="#FLG033"  Part="1"
-AR Path="/5978A36B/5978B8AA/599195CA" Ref="#FLG080"  Part="1"
-F 0 "#FLG080" H 3800 3575 50  0001 C CNN
+AR Path="/597003E2/597189AE/599195CA" Ref="#FLG601"  Part="1"
+AR Path="/5978A36B/5978B8AA/599195CA" Ref="#FLG3001"  Part="1"
+F 0 "#FLG3001" H 3800 3575 50  0001 C CNN
 F 1 "PWR_FLAG" H 3800 3650 50  0000 C CNN
 F 2 "" H 3800 3500 50  0001 C CNN
