File: electrical/ECU/kicad_ECU/ATmega256RFR2.sch (KiCad schematic (older format))
At the start: 30 parts, among them CON3 AVR-ISP-6, J5 FTDI, SW2 SW_Push_Dual, U18 SI8620BC-B-IS, U19 ATmega256RFR2, Y3 16MHz, Y4 ABS07AIG

Commit message: minor naming change
Parts:
- renumbered C51 to C2401, C52 to C2402, C53 to C2403, C54 to C2404, C55 to C2405, C56 to C2406, C57 to C2407, C58 to C2408, C59 to C2409, C60 to C2410, C61 to C2411, C62 to C2412, C63 to C2413, CON3 to CON2401, D35 to D2401, D36 to D2402, D37 to D2403, J5 to J2401, L7 to L2401, R54 to R2401, R55 to R2402, R56 to R2403, R57 to R2404, R58 to R2405, R59 to R2406, SW2 to SW2401, U18 to U2401, U19 to U2402, Y3 to Y2401, Y4 to Y2402
Changed lines of the file:
@@
 $EndDescr
 $Comp
-L ATmega256RFR2 U19
+L ATmega256RFR2 U2402
 U 1 1 5978B75B
 P 4700 4950
-F 0 "U19" H 4700 4800 60  0000 C CNN
+F 0 "U2402" H 4700 4800 60  0000 C CNN
 F 1 "ATmega256RFR2" H 4700 5050 60  0000 C CNN
 F 2 "" H 4700 4950 60  0000 C CNN
@@
 $EndComp
 $Comp
-L C C61
+L C C2411
 U 1 1 5978B762
 P 5850 2400
-F 0 "C61" H 5875 2500 50  0000 L CNN
+F 0 "C2411" H 5875 2500 50  0000 L CNN
 F 1 "100n" H 5875 2300 50  0000 L CNN
 F 2 "" H 5888 2250 50  0001 C CNN
@@
 $EndComp
 $Comp
-L C C60
+L C C2410
 U 1 1 5978B769
 P 5550 2400
-F 0 "C60" H 5575 2500 50  0000 L CNN
+F 0 "C2410" H 5575 2500 50  0000 L CNN
 F 1 "100n" H 5575 2300 50  0000 L CNN
 F 2 "" H 5588 2250 50  0001 C CNN
@@
 $EndComp
 $Comp
-L C C59
+L C C2409
 U 1 1 5978B770
 P 5250 2400
-F 0 "C59" H 5275 2500 50  0000 L CNN
+F 0 "C2409" H 5275 2500 50  0000 L CNN
 F 1 "100n" H 5275 2300 50  0000 L CNN
 F 2 "" H 5288 2250 50  0001 C CNN
@@
 $EndComp
 $Comp
-L C C62
+L C C2412
 U 1 1 5978B777
 P 6150 2400
-F 0 "C62" H 6175 2500 50  0000 L CNN
+F 0 "C2412" H 6175 2500 50  0000 L CNN
 F 1 "100n" H 6175 2300 50  0000 L CNN
 F 2 "" H 6188 2250 50  0001 C CNN
@@
 $EndComp
 $Comp
-L Earth #PWR064
+L Earth #PWR2405
 U 1 1 5978B77E
 P 5550 2800
-F 0 "#PWR064" H 5550 2550 50  0001 C CNN
+F 0 "#PWR2405" H 5550 2550 50  0001 C CNN
 F 1 "Earth" H 5550 2650 50  0001 C CNN
 F 2 "" H 5550 2800 50  0001 C CNN
@@
 $EndComp
 $Comp
-L Crystal Y3
+L Crystal Y2401
 U 1 1 5978B78A
 P 1900 5000
-F 0 "Y3" H 1900 5150 50  0000 C CNN
+F 0 "Y2401" H 1900 5150 50  0000 C CNN
 F 1 "16MHz" H 1900 4850 50  0000 C CNN
 F 2 "" H 1900 5000 60  0000 C CNN
@@
 $EndComp
 $Comp
-L C C51
+L C C2401
 U 1 1 5978B791
 P 1500 4850
-F 0 "C51" H 1525 4950 50  0000 L CNN
+F 0 "C2401" H 1525 4950 50  0000 L CNN
 F 1 "10pF" H 1525 4750 50  0000 L CNN
 F 2 "" H 1538 4700 30  0000 C CNN
@@
 $EndComp
 $Comp
-L C C52
+L C C2402
 U 1 1 5978B798
 P 1500 5150
-F 0 "C52" H 1525 5250 50  0000 L CNN
+F 0 "C2402" H 1525 5250 50  0000 L CNN
 F 1 "10pF" H 1525 5050 50  0000 L CNN
 F 2 "" H 1538 5000 30  0000 C CNN
@@
 $EndComp
 $Comp
-L R R54
+L R R2401
 U 1 1 5978B79F
 P 900 5000
-F 0 "R54" V 1000 5000 50  0000 C CNN
+F 0 "R2401" V 1000 5000 50  0000 C CNN
 F 1 "1M" V 900 5000 50  0000 C CNN
 F 2 "" V 830 5000 30  0000 C CNN
@@
 $EndComp
 $Comp
-L C C58
+L C C2408
 U 1 1 5978B7AC
 P 3100 7100
-F 0 "C58" H 3125 7200 50  0000 L CNN
+F 0 "C2408" H 3125 7200 50  0000 L CNN
 F 1 "1uF" H 3125 7000 50  0000 L CNN
 F 2 "" H 3138 6950 50  0001 C CNN
@@
 $EndComp
 $Comp
-L C C56
+L C C2406
 U 1 1 5978B7B3
 P 2450 7100
-F 0 "C56" H 2475 7200 50  0000 L CNN
+F 0 "C2406" H 2475 7200 50  0000 L CNN
 F 1 "1uF" H 2475 7000 50  0000 L CNN
 F 2 "" H 2488 6950 50  0001 C CNN
@@
 $EndComp
 $Comp
-L R R57
+L R R2404
 U 1 1 5978B7C6
 P 2000 7100
-F 0 "R57" V 2080 7100 50  0000 C CNN
+F 0 "R2404" V 2080 7100 50  0000 C CNN
 F 1 "10k" V 2000 7100 50  0000 C CNN
 F 2 "" V 1930 7100 50  0001 C CNN
@@
 $EndComp
 $Comp
-L R R55
+L R R2402
 U 1 1 5978B7CD
 P 1600 7100
-F 0 "R55" V 1680 7100 50  0000 C CNN
+F 0 "R2402" V 1680 7100 50  0000 C CNN
 F 1 "10k" V 1600 7100 50  0000 C CNN
 F 2 "" V 1530 7100 50  0001 C CNN
@@
 CLKI
 $Comp
-L Crystal Y4
+L Crystal Y2402
 U 1 1 5978B7E1
 P 2700 5850
-F 0 "Y4" H 2700 6000 50  0000 C CNN
+F 0 "Y2402" H 2700 6000 50  0000 C CNN
 F 1 "ABS07AIG" H 2700 5700 50  0000 C CNN
 F 2 "" H 2700 5850 60  0000 C CNN
@@
 $EndComp
 $Comp
-L C C53
+L C C2403
 U 1 1 5978B7E8
 P 2300 5700
-F 0 "C53" H 2325 5800 50  0000 L CNN
+F 0 "C2403" H 2325 5800 50  0000 L CNN
 F 1 "10pF" H 2325 5600 50  0000 L CNN
 F 2 "" H 2338 5550 30  0000 C CNN
@@
 $EndComp
 $Comp
-L C C54
+L C C2404
 U 1 1 5978B7EF
 P 2300 6000
-F 0 "C54" H 2325 6100 50  0000 L CNN
+F 0 "C2404" H 2325 6100 50  0000 L CNN
 F 1 "10pF" H 2325 5900 50  0000 L CNN
 F 2 "" H 2338 5850 30  0000 C CNN
@@
 $EndComp
 $Comp
-L R R56
+L R R2403
 U 1 1 5978B7F6
 P 1700 5850
-F 0 "R56" V 1800 5850 50  0000 C CNN
+F 0 "R2403" V 1800 5850 50  0000 C CNN
 F 1 "10M" V 1700 5850 50  0000 C CNN
 F 2 "" V 1630 5850 30  0000 C CNN
@@
 RFN
 $Comp
-L AVR-ISP-6 CON3
+L AVR-ISP-6 CON2401
 U 1 1 5978B82F
 P 1750 1200
-F 0 "CON3" H 1645 1440 50  0000 C CNN
+F 0 "CON2401" H 1645 1440 50  0000 C CNN
 F 1 "AVR-ISP-6" H 1485 970 50  0000 L BNN
 F 2 "AVR-ISP-6" V 1230 1240 50  0001 C CNN
@@
 MOSI
 $Comp
-L CONN_01X06 J5
+L CONN_01X06 J2401
 U 1 1 5978B843
 P 1650 2350
-F 0 "J5" H 1650 2700 50  0000 C CNN
+F 0 "J2401" H 1650 2700 50  0000 C CNN
 F 1 "FTDI" V 1750 2350 50  0000 C CNN
 F 2 "" H 1650 2350 50  0001 C CNN
@@
 RESET
 $Comp
-L R R58
+L R R2405
 U 1 1 5978B8C4
 P 2400 3350
-F 0 "R58" V 2480 3350 50  0000 C CNN
+F 0 "R2405" V 2480 3350 50  0000 C CNN
 F 1 "10K" V 2400 3350 50  0000 C CNN
 F 2 "" V 2330 3350 50  0001 C CNN
@@
 VCC
 $Comp
-L Ferrite_Bead L7
+L Ferrite_Bead L2401
 U 1 1 5978B8CC
 P 10450 4800
-F 0 "L7" V 10300 4825 50  0000 C CNN
+F 0 "L2401" V 10300 4825 50  0000 C CNN
 F 1 "Ferrite_Bead" V 10600 4800 50  0000 C CNN
 F 2 "" V 10380 4800 50  0001 C CNN
@@
 $EndComp
 $Comp
-L CP1 C63
+L CP1 C2413
 U 1 1 5978B8D3
 P 10450 5450
-F 0 "C63" H 10475 5550 50  0000 L CNN
+F 0 "C2413" H 10475 5550 50  0000 L CNN
 F 1 "4.7uF/10v" H 10475 5350 50  0000 L CNN
 F 2 "" H 10450 5450 50  0001 C CNN
@@
 $EndComp
 $Comp
-L R R59
+L R R2406
 U 1 1 5978B8E0
 P 10850 5450
-F 0 "R59" V 10930 5450 50  0000 C CNN
+F 0 "R2406" V 10930 5450 50  0000 C CNN
 F 1 "330" V 10850 5450 50  0000 C CNN
 F 2 "" V 10780 5450 50  0001 C CNN
@@
 $EndComp
 $Comp
-L LED-RESCUE-airhead_ecu D37
+L LED-RESCUE-airhead_ecu D2403
 U 1 1 5978B8E7
 P 10850 5900
-F 0 "D37" H 10850 6000 50  0000 C CNN
+F 0 "D2403" H 10850 6000 50  0000 C CNN
 F 1 "GREEN" H 10850 5800 50  0000 C CNN
 F 2 "" H 10850 5900 50  0001 C CNN
@@
 B3
 $Comp
-L C C55
+L C C2405
 U 1 1 5978B9E6
 P 2400 3650
-F 0 "C55" H 2425 3750 50  0000 L CNN
+F 0 "C2405" H 2425 3750 50  0000 L CNN
 F 1 "22pF" H 2425 3550 50  0000 L CNN
 F 2 "" H 2438 3500 50  0001 C CNN
@@
 HC
 $Comp
-L SI8620BC-B-IS U18
+L SI8620BC-B-IS U2401
 U 1 1 5978F344
 P 4250 950
-F 0 "U18" H 4250 850 50  0000 C CNN
+F 0 "U2401" H 4250 850 50  0000 C CNN
 F 1 "SI8620BC-B-IS" H 4250 1050 50  0000 C CNN
 F 2 "MODULE" H 4250 950 50  0001 C CNN
@@
 points_in
 $Comp
-L Earth #PWR065
+L Earth #PWR2402
 U 1 1 5978F513
 P 3500 1300
-F 0 "#PWR065" H 3500 1050 50  0001 C CNN
+F 0 "#PWR2402" H 3500 1050 50  0001 C CNN
 F 1 "Earth" H 3500 1150 50  0001 C CNN
 F 2 "" H 3500 1300 50  0001 C CNN
@@
 $EndComp
 $Comp
-L Earth #PWR066
+L Earth #PWR2403
 U 1 1 5978F571
 P 5000 1300
-F 0 "#PWR066" H 5000 1050 50  0001 C CNN
+F 0 "#PWR2403" H 5000 1050 50  0001 C CNN
 F 1 "Earth" H 5000 1150 50  0001 C CNN
 F 2 "" H 5000 1300 50  0001 C CNN
@@
 TACH2
 $Comp
-L D D35
+L D D2401
 U 1 1 597D4967
 P 6400 7350
-F 0 "D35" H 6400 7450 50  0000 C CNN
+F 0 "D2401" H 6400 7450 50  0000 C CNN
 F 1 "D" H 6400 7250 50  0000 C CNN
 F 2 "" H 6400 7350 50  0001 C CNN
@@
 C2
 $Comp
-L D D36
+L D D2402
 U 1 1 597D548E
 P 6400 7500
-F 0 "D36" H 6400 7600 50  0000 C CNN
+F 0 "D2402" H 6400 7600 50  0000 C CNN
 F 1 "D" H 6400 7400 50  0000 C CNN
 F 2 "" H 6400 7500 50  0001 C CNN
@@
 NoConn ~ 3100 3200
 $Comp
-L SW_Push_Dual SW2
+L SW_Push_Dual SW2401
 U 1 1 597D7A8C
 P 1950 3850
-F 0 "SW2" H 2000 3950 50  0000 L CNN
+F 0 "SW2401" H 2000 3950 50  0000 L CNN
 F 1 "SW_Push_Dual" H 1950 3580 50  0000 C CNN
 F 2 "" H 1950 4050 50  0001 C CNN
@@
 $EndSheet
 $Comp
-L PWR_FLAG #FLG067
+L PWR_FLAG #FLG2401
 U 1 1 5991997C
 P 10850 4950
-F 0 "#FLG067" H 10850 5025 50  0001 C CNN
+F 0 "#FLG2401" H 10850 5025 50  0001 C CNN
 F 1 "PWR_FLAG" H 10850 5100 50  0000 C CNN
 F 2 "" H 10850 4950 50  0001 C CNN
@@
 Connection ~ 10850 4950
 $Comp
-L C C57
+L C C2407
 U 1 1 5991A507
 P 2800 7100
-F 0 "C57" H 2825 7200 50  0000 L CNN
+F 0 "C2407" H 2825 7200 50  0000 L CNN
 F 1 "1uF" H 2825 7000 50  0000 L CNN
 F 2 "" H 2838 6950 50  0001 C CNN
@@
 Connection ~ 1600 7350
 $Comp
-L Earth #PWR068
+L Earth #PWR2406
 U 1 1 5992AD41
 P 10450 6250
-F 0 "#PWR068" H 10450 6000 50  0001 C CNN
+F 0 "#PWR2406" H 10450 6000 50  0001 C CNN
 F 1 "Earth" H 10450 6100 50  0001 C CNN
 F 2 "" H 10450 6250 50  0001 C CNN
@@
 Connection ~ 10450 6150
 $Comp
-L Earth #PWR069
+L Earth #PWR2404
 U 1 1 5992DD60
 P 5050 7550
-F 0 "#PWR069" H 5050 7300 50  0001 C CNN
+F 0 "#PWR2404" H 5050 7300 50  0001 C CNN
 F 1 "Earth" H 5050 7400 50  0001 C CNN
 F 2 "" H 5050 7550 50  0001 C CNN
@@
 Connection ~ 1050 6100
 $Comp
-L Earth #PWR070
+L Earth #PWR2401
 U 1 1 5993EE4E
 P 2250 1500
-F 0 "#PWR070" H 2250 1250 50  0001 C CNN
+F 0 "#PWR2401" H 2250 1250 50  0001 C CNN
 F 1 "Earth" H 2250 1350 50  0001 C CNN
 F 2 "" H 2250 1500 50  0001 C CNN
