File: electrical/ECU/kicad_ECU/ATmega256RFR2_Conn.sch (KiCad schematic (older format))
At the start: 54 parts, among them CON1 AVR-ISP-6, CON2 AVR-JTAG-10, J2 FTDI, J3 CONN_01X15, J4 CONN_01X15

Commit message: minor naming change
Parts:
- renumbered CON1 to CON901, CON2 to CON902, D6 to D901, D7 to D902, D8 to D903, D9 to D904, D10 to D905, D11 to D906, D12 to D907, D13 to D908, D14 to D909, D15 to D910, D16 to D911, D17 to D912, D18 to D913, D19 to D914, D20 to D915, D21 to D916, D22 to D917, D23 to D918, D24 to D919, D25 to D920, D26 to D921, D27 to D922, D28 to D923, D29 to D924, D30 to D925, F3 to F901, F4 to F902, F5 to F903, F6 to F904, F7 to F905, F8 to F906, F9 to F907, F10 to F908, F11 to F909, F12 to F910, F13 to F911, F14 to F912, F15 to F913, F16 to F914, F17 to F915, F18 to F916, F19 to F917, F20 to F918, F21 to F919, F22 to F920, F23 to F921, F24 to F922, F25 to F923, F26 to F924, J2 to J901, J3 to J902, J4 to J903
