File: electrical/ECU/kicad_ECU/ATmega256RFR2_USB.sch (KiCad schematic (older format))
At the start: 30 parts, among them SW1 SW_Push, U5 ATmega256RFR2, Y1 16MHz, Y2 ABS07AIG

Commit message: minor naming change
Parts:
- renumbered C1 to C401, C2 to C402, C3 to C403, C4 to C404, C5 to C405, C6 to C406, C7 to C407, C8 to C408, C9 to C409, C10 to C410, C11 to C411, C12 to C412, C13 to C413, D1 to D401, L2 to L401, R6 to R401, R7 to R402, R8 to R403, R9 to R404, R10 to R405, R11 to R406, R12 to R407, R13 to R408, R14 to R409, R15 to R410, R16 to R411, SW1 to SW401, U5 to U401, Y1 to Y401, Y2 to Y402
Changed lines of the file:
@@
 $EndDescr
 $Comp
-L R R7
+L R R402
 U 1 1 59702EEA
 P 1250 1200
-F 0 "R7" V 1330 1200 50  0000 C CNN
+F 0 "R402" V 1330 1200 50  0000 C CNN
 F 1 "10k" V 1250 1200 50  0000 C CNN
 F 2 "" V 1180 1200 30  0000 C CNN
@@
 $EndComp
 $Comp
-L R R12
+L R R407
 U 1 1 59702EF1
 P 1550 1200
-F 0 "R12" V 1630 1200 50  0000 C CNN
+F 0 "R407" V 1630 1200 50  0000 C CNN
 F 1 "10k" V 1550 1200 50  0000 C CNN
 F 2 "" V 1480 1200 30  0000 C CNN
@@
 SCL
 $Comp
-L R R8
+L R R403
 U 1 1 59702F2F
 P 1250 1200
-F 0 "R8" V 1330 1200 50  0000 C CNN
+F 0 "R403" V 1330 1200 50  0000 C CNN
 F 1 "10k" V 1250 1200 50  0000 C CNN
 F 2 "" V 1180 1200 30  0000 C CNN
@@
 $EndComp
 $Comp
-L R R13
+L R R408
 U 1 1 59702F36
 P 1550 1200
-F 0 "R13" V 1630 1200 50  0000 C CNN
+F 0 "R408" V 1630 1200 50  0000 C CNN
 F 1 "10k" V 1550 1200 50  0000 C CNN
 F 2 "" V 1480 1200 30  0000 C CNN
@@
 SCL
 $Comp
-L ATmega256RFR2 U5
+L ATmega256RFR2 U401
 U 1 1 59702F40
 P 4450 3550
-F 0 "U5" H 4450 3400 60  0000 C CNN
+F 0 "U401" H 4450 3400 60  0000 C CNN
 F 1 "ATmega256RFR2" H 4450 3650 60  0000 C CNN
 F 2 "" H 4450 3550 60  0000 C CNN
@@
 $EndComp
 $Comp
-L C C11
+L C C411
 U 1 1 59702F47
 P 5600 1000
-F 0 "C11" H 5625 1100 50  0000 L CNN
+F 0 "C411" H 5625 1100 50  0000 L CNN
 F 1 "100n" H 5625 900 50  0000 L CNN
 F 2 "" H 5638 850 50  0001 C CNN
@@
 $EndComp
 $Comp
-L C C10
+L C C410
 U 1 1 59702F4E
 P 5300 1000
-F 0 "C10" H 5325 1100 50  0000 L CNN
+F 0 "C410" H 5325 1100 50  0000 L CNN
 F 1 "100n" H 5325 900 50  0000 L CNN
 F 2 "" H 5338 850 50  0001 C CNN
@@
 $EndComp
 $Comp
-L C C9
+L C C409
 U 1 1 59702F55
 P 5000 1000
-F 0 "C9" H 5025 1100 50  0000 L CNN
+F 0 "C409" H 5025 1100 50  0000 L CNN
 F 1 "100n" H 5025 900 50  0000 L CNN
 F 2 "" H 5038 850 50  0001 C CNN
@@
 $EndComp
 $Comp
-L C C12
+L C C412
 U 1 1 59702F5C
 P 5900 1000
-F 0 "C12" H 5925 1100 50  0000 L CNN
+F 0 "C412" H 5925 1100 50  0000 L CNN
 F 1 "100n" H 5925 900 50  0000 L CNN
 F 2 "" H 5938 850 50  0001 C CNN
@@
 $EndComp
 $Comp
-L Earth #PWR019
+L Earth #PWR405
 U 1 1 59702F63
 P 5300 1400
-F 0 "#PWR019" H 5300 1150 50  0001 C CNN
+F 0 "#PWR405" H 5300 1150 50  0001 C CNN
 F 1 "Earth" H 5300 1250 50  0001 C CNN
 F 2 "" H 5300 1400 50  0001 C CNN
@@
 $EndComp
 $Comp
-L Earth #PWR020
+L Earth #PWR404
 U 1 1 59702F6A
 P 4900 6350
-F 0 "#PWR020" H 4900 6100 50  0001 C CNN
+F 0 "#PWR404" H 4900 6100 50  0001 C CNN
 F 1 "Earth" H 4900 6200 50  0001 C CNN
 F 2 "" H 4900 6350 50  0001 C CNN
@@
 $EndComp
 $Comp
-L Crystal Y1
+L Crystal Y401
 U 1 1 59702F70
 P 1650 3600
-F 0 "Y1" H 1650 3750 50  0000 C CNN
+F 0 "Y401" H 1650 3750 50  0000 C CNN
 F 1 "16MHz" H 1650 3450 50  0000 C CNN
 F 2 "" H 1650 3600 60  0000 C CNN
@@
 $EndComp
 $Comp
-L C C1
+L C C401
 U 1 1 59702F77
 P 1250 3450
-F 0 "C1" H 1275 3550 50  0000 L CNN
+F 0 "C401" H 1275 3550 50  0000 L CNN
 F 1 "10pF" H 1275 3350 50  0000 L CNN
 F 2 "" H 1288 3300 30  0000 C CNN
@@
 $EndComp
 $Comp
-L C C2
+L C C402
 U 1 1 59702F7E
 P 1250 3750
-F 0 "C2" H 1275 3850 50  0000 L CNN
+F 0 "C402" H 1275 3850 50  0000 L CNN
 F 1 "10pF" H 1275 3650 50  0000 L CNN
 F 2 "" H 1288 3600 30  0000 C CNN
@@
 $EndComp
 $Comp
-L R R6
+L R R401
 U 1 1 59702F85
 P 650 3600
-F 0 "R6" V 750 3600 50  0000 C CNN
+F 0 "R401" V 750 3600 50  0000 C CNN
 F 1 "1M" V 650 3600 50  0000 C CNN
 F 2 "" V 580 3600 30  0000 C CNN
@@
 $EndComp
 $Comp
-L Earth #PWR021
+L Earth #PWR401
 U 1 1 59702F8C
 P 900 3750
-F 0 "#PWR021" H 900 3500 50  0001 C CNN
+F 0 "#PWR401" H 900 3500 50  0001 C CNN
 F 1 "Earth" H 900 3600 50  0001 C CNN
 F 2 "" H 900 3750 50  0001 C CNN
@@
 $EndComp
 $Comp
-L C C8
+L C C408
 U 1 1 59702F92
 P 2850 5700
-F 0 "C8" H 2875 5800 50  0000 L CNN
+F 0 "C408" H 2875 5800 50  0000 L CNN
 F 1 "1uF" H 2875 5600 50  0000 L CNN
 F 2 "" H 2888 5550 50  0001 C CNN
@@
 $EndComp
 $Comp
-L C C6
+L C C406
 U 1 1 59702F99
 P 2200 5700
-F 0 "C6" H 2225 5800 50  0000 L CNN
+F 0 "C406" H 2225 5800 50  0000 L CNN
 F 1 "1uF" H 2225 5600 50  0000 L CNN
 F 2 "" H 2238 5550 50  0001 C CNN
@@
 $EndComp
 $Comp
-L R R14
+L R R409
 U 1 1 59702FAC
 P 1750 5700
-F 0 "R14" V 1830 5700 50  0000 C CNN
+F 0 "R409" V 1830 5700 50  0000 C CNN
 F 1 "10k" V 1750 5700 50  0000 C CNN
 F 2 "" V 1680 5700 50  0001 C CNN
@@
 $EndComp
 $Comp
-L R R9
+L R R404
 U 1 1 59702FB3
 P 1350 5700
-F 0 "R9" V 1430 5700 50  0000 C CNN
+F 0 "R404" V 1430 5700 50  0000 C CNN
 F 1 "10k" V 1350 5700 50  0000 C CNN
 F 2 "" V 1280 5700 50  0001 C CNN
@@
 CLKI
 $Comp
-L Crystal Y2
+L Crystal Y402
 U 1 1 59702FC7
 P 2450 4450
-F 0 "Y2" H 2450 4600 50  0000 C CNN
+F 0 "Y402" H 2450 4600 50  0000 C CNN
 F 1 "ABS07AIG" H 2450 4300 50  0000 C CNN
 F 2 "" H 2450 4450 60  0000 C CNN
@@
 $EndComp
 $Comp
-L C C3
+L C C403
 U 1 1 59702FCE
 P 2050 4300
-F 0 "C3" H 2075 4400 50  0000 L CNN
+F 0 "C403" H 2075 4400 50  0000 L CNN
 F 1 "10pF" H 2075 4200 50  0000 L CNN
 F 2 "" H 2088 4150 30  0000 C CNN
@@
 $EndComp
 $Comp
-L C C4
+L C C404
 U 1 1 59702FD5
 P 2050 4600
-F 0 "C4" H 2075 4700 50  0000 L CNN
+F 0 "C404" H 2075 4700 50  0000 L CNN
 F 1 "10pF" H 2075 4500 50  0000 L CNN
 F 2 "" H 2088 4450 30  0000 C CNN
@@
 $EndComp
 $Comp
-L R R11
+L R R406
 U 1 1 59702FDC
 P 1450 4450
-F 0 "R11" V 1550 4450 50  0000 C CNN
+F 0 "R406" V 1550 4450 50  0000 C CNN
 F 1 "10M" V 1450 4450 50  0000 C CNN
 F 2 "" V 1380 4450 30  0000 C CNN
@@
 $EndComp
 $Comp
-L Earth #PWR022
+L Earth #PWR403
 U 1 1 59702FE3
 P 1700 4600
-F 0 "#PWR022" H 1700 4350 50  0001 C CNN
+F 0 "#PWR403" H 1700 4350 50  0001 C CNN
 F 1 "Earth" H 1700 4450 50  0001 C CNN
 F 2 "" H 1700 4600 50  0001 C CNN
@@
 RESET
 $Comp
-L R R15
+L R R410
 U 1 1 5972503B
 P 2150 1950
-F 0 "R15" V 2230 1950 50  0000 C CNN
+F 0 "R410" V 2230 1950 50  0000 C CNN
 F 1 "10K" V 2150 1950 50  0000 C CNN
 F 2 "" V 2080 1950 50  0001 C CNN
@@
 VCC
 $Comp
-L Ferrite_Bead L2
+L Ferrite_Bead L401
 U 1 1 597260BD
 P 10050 4800
-F 0 "L2" V 9900 4825 50  0000 C CNN
+F 0 "L401" V 9900 4825 50  0000 C CNN
 F 1 "Ferrite_Bead" V 10200 4800 50  0000 C CNN
 F 2 "" V 9980 4800 50  0001 C CNN
@@
 $EndComp
 $Comp
-L CP1 C13
+L CP1 C413
 U 1 1 597262C3
 P 10050 5450
-F 0 "C13" H 10075 5550 50  0000 L CNN
+F 0 "C413" H 10075 5550 50  0000 L CNN
 F 1 "4.7uF/10v" H 10075 5350 50  0000 L CNN
 F 2 "" H 10050 5450 50  0001 C CNN
@@
 $EndComp
 $Comp
-L R R16
+L R R411
 U 1 1 59727C19
 P 10450 5450
-F 0 "R16" V 10530 5450 50  0000 C CNN
+F 0 "R411" V 10530 5450 50  0000 C CNN
 F 1 "330" V 10450 5450 50  0000 C CNN
 F 2 "" V 10380 5450 50  0001 C CNN
@@
 $EndComp
 $Comp
-L LED-RESCUE-airhead_ecu D1
+L LED-RESCUE-airhead_ecu D401
 U 1 1 59727E25
 P 10450 5900
-F 0 "D1" H 10450 6000 50  0000 C CNN
+F 0 "D401" H 10450 6000 50  0000 C CNN
 F 1 "GREEN" H 10450 5800 50  0000 C CNN
 F 2 "" H 10450 5900 50  0001 C CNN
@@
 $EndComp
 $Comp
-L Earth #PWR023
+L Earth #PWR407
 U 1 1 59727F26
 P 10450 6300
-F 0 "#PWR023" H 10450 6050 50  0001 C CNN
+F 0 "#PWR407" H 10450 6050 50  0001 C CNN
 F 1 "Earth" H 10450 6150 50  0001 C CNN
 F 2 "" H 10450 6300 50  0001 C CNN
@@
 $EndComp
 $Comp
-L SW_Push SW1
+L SW_Push SW401
 U 1 1 5972882F
 P 1700 2350
-F 0 "SW1" H 1750 2450 50  0000 L CNN
+F 0 "SW401" H 1750 2450 50  0000 L CNN
 F 1 "SW_Push" H 1700 2290 50  0000 C CNN
 F 2 "" H 1700 2550 50  0001 C CNN
@@
 $EndComp
 $Comp
-L Earth #PWR024
+L Earth #PWR402
 U 1 1 5972890E
 P 1700 2800
-F 0 "#PWR024" H 1700 2550 50  0001 C CNN
+F 0 "#PWR402" H 1700 2550 50  0001 C CNN
 F 1 "Earth" H 1700 2650 50  0001 C CNN
 F 2 "" H 1700 2800 50  0001 C CNN
@@
 PG5
 $Comp
-L C C5
+L C C405
 U 1 1 5972ECDE
 P 2150 2250
-F 0 "C5" H 2175 2350 50  0000 L CNN
+F 0 "C405" H 2175 2350 50  0000 L CNN
 F 1 "22pF" H 2175 2150 50  0000 L CNN
 F 2 "" H 2188 2100 50  0001 C CNN
@@
 $EndSheet
 $Comp
-L Earth #PWR025
+L Earth #PWR406
 U 1 1 59819988
 P 8350 6200
-F 0 "#PWR025" H 8350 5950 50  0001 C CNN
+F 0 "#PWR406" H 8350 5950 50  0001 C CNN
 F 1 "Earth" H 8350 6050 50  0001 C CNN
 F 2 "" H 8350 6200 50  0001 C CNN
@@
 	11000 2550 10650 2550
 $Comp
-L R R10
+L R R405
 U 1 1 598DD98E
 P 1400 2100
-F 0 "R10" V 1480 2100 50  0000 C CNN
+F 0 "R405" V 1480 2100 50  0000 C CNN
 F 1 "1k" V 1400 2100 50  0000 C CNN
 F 2 "" V 1330 2100 50  0001 C CNN
@@
 NoConn ~ 2500 1800
 $Comp
-L PWR_FLAG #FLG026
+L PWR_FLAG #FLG401
 U 1 1 5990E997
 P 4800 700
-F 0 "#FLG026" H 4800 775 50  0001 C CNN
+F 0 "#FLG401" H 4800 775 50  0001 C CNN
 F 1 "PWR_FLAG" H 4800 850 50  0000 C CNN
 F 2 "" H 4800 700 50  0001 C CNN
@@
 	11000 2250 10650 2250
 $Comp
-L C C7
+L C C407
 U 1 1 599167D8
 P 2550 5700
-F 0 "C7" H 2575 5800 50  0000 L CNN
+F 0 "C407" H 2575 5800 50  0000 L CNN
 F 1 "1uF" H 2575 5600 50  0000 L CNN
 F 2 "" H 2588 5550 50  0001 C CNN
