File: electrical/ECU/kicad_ECU/BRV.sch (KiCad schematic (older format))
At the start: 5 parts

Commit message: minor naming change
Parts:
- renumbered C49 to C2301, C50 to C2302, R51 to R2301, R52 to R2302, R53 to R2303
Changed lines of the file:
@@
 12v
 $Comp
-L R R51
+L R R2301
 U 1 1 59783EC3
 P 5000 3250
-F 0 "R51" V 5080 3250 50  0000 C CNN
+F 0 "R2301" V 5080 3250 50  0000 C CNN
 F 1 "3.9k" V 5000 3250 50  0000 C CNN
 F 2 "" V 4930 3250 50  0001 C CNN
@@
 $EndComp
 $Comp
-L R R52
+L R R2302
 U 1 1 59783EE2
 P 5000 3900
-F 0 "R52" V 5080 3900 50  0000 C CNN
+F 0 "R2302" V 5080 3900 50  0000 C CNN
 F 1 "1k" V 5000 3900 50  0000 C CNN
 F 2 "" V 4930 3900 50  0001 C CNN
@@
 $EndComp
 $Comp
-L C C49
+L C C2301
 U 1 1 59783F06
 P 5550 3900
-F 0 "C49" H 5575 4000 50  0000 L CNN
+F 0 "C2301" H 5575 4000 50  0000 L CNN
 F 1 "0.1uF" H 5575 3800 50  0000 L CNN
 F 2 "" H 5588 3750 50  0001 C CNN
@@
 $EndComp
 $Comp
-L C C50
+L C C2302
 U 1 1 59783F32
 P 6650 3900
-F 0 "C50" H 6675 4000 50  0000 L CNN
+F 0 "C2302" H 6675 4000 50  0000 L CNN
 F 1 "0.22uF" H 6675 3800 50  0000 L CNN
 F 2 "" H 6688 3750 50  0001 C CNN
@@
 $EndComp
 $Comp
-L R R53
+L R R2303
 U 1 1 59783F66
 P 5950 3550
-F 0 "R53" V 6030 3550 50  0000 C CNN
+F 0 "R2303" V 6030 3550 50  0000 C CNN
 F 1 "470" V 5950 3550 50  0000 C CNN
 F 2 "" V 5880 3550 50  0001 C CNN
@@
 Connection ~ 6650 3550
 $Comp
-L Earth #PWR063
+L Earth #PWR2301
 U 1 1 59784002
 P 6650 4350
-F 0 "#PWR063" H 6650 4100 50  0001 C CNN
+F 0 "#PWR2301" H 6650 4100 50  0001 C CNN
 F 1 "Earth" H 6650 4200 50  0001 C CNN
 F 2 "" H 6650 4350 50  0001 C CNN
