File: electrical/ECU/kicad_ECU/TPS.sch (KiCad schematic (older format))
At the start: 3 parts

Commit message: minor naming change
Parts:
- renumbered C33 to C1501, C34 to C1502, R33 to R1501
Changed lines of the file:
@@
 CPU
 $Comp
-L R R33
+L R R1501
 U 1 1 597755F5
 P 5700 3150
-AR Path="/5974D512/5977551F/597755F5" Ref="R33"  Part="1"
-AR Path="/5974D512/59775648/597755F5" Ref="R34"  Part="1"
-F 0 "R34" V 5780 3150 50  0000 C CNN
+AR Path="/5974D512/5977551F/597755F5" Ref="R1501"  Part="1"
+AR Path="/5974D512/59775648/597755F5" Ref="R1601"  Part="1"
+F 0 "R1601" V 5780 3150 50  0000 C CNN
 F 1 "470" V 5700 3150 50  0000 C CNN
 F 2 "" V 5630 3150 50  0001 C CNN
@@
 $EndComp
 $Comp
-L C C33
+L C C1501
 U 1 1 597755FC
 P 5200 3550
-AR Path="/5974D512/5977551F/597755FC" Ref="C33"  Part="1"
-AR Path="/5974D512/59775648/597755FC" Ref="C35"  Part="1"
-F 0 "C35" H 5225 3650 50  0000 L CNN
+AR Path="/5974D512/5977551F/597755FC" Ref="C1501"  Part="1"
+AR Path="/5974D512/59775648/597755FC" Ref="C1601"  Part="1"
+F 0 "C1601" H 5225 3650 50  0000 L CNN
 F 1 "0.1uF" H 5225 3450 50  0000 L CNN
 F 2 "" H 5238 3400 50  0001 C CNN
@@
 $EndComp
 $Comp
-L C C34
+L C C1502
 U 1 1 59775603
 P 6700 3550
-AR Path="/5974D512/5977551F/59775603" Ref="C34"  Part="1"
-AR Path="/5974D512/59775648/59775603" Ref="C36"  Part="1"
-F 0 "C36" H 6725 3650 50  0000 L CNN
+AR Path="/5974D512/5977551F/59775603" Ref="C1502"  Part="1"
+AR Path="/5974D512/59775648/59775603" Ref="C1602"  Part="1"
+F 0 "C1602" H 6725 3650 50  0000 L CNN
 F 1 "0.22uF" H 6725 3450 50  0000 L CNN
 F 2 "" H 6738 3400 50  0001 C CNN
@@
 $EndComp
 $Comp
-L Earth #PWR054
+L Earth #PWR1501
 U 1 1 5977560A
 P 6700 4200
-AR Path="/5974D512/5977551F/5977560A" Ref="#PWR054"  Part="1"
-AR Path="/5974D512/59775648/5977560A" Ref="#PWR055"  Part="1"
-F 0 "#PWR055" H 6700 3950 50  0001 C CNN
+AR Path="/5974D512/5977551F/5977560A" Ref="#PWR1501"  Part="1"
+AR Path="/5974D512/59775648/5977560A" Ref="#PWR1601"  Part="1"
+F 0 "#PWR1601" H 6700 3950 50  0001 C CNN
 F 1 "Earth" H 6700 4050 50  0001 C CNN
 F 2 "" H 6700 4200 50  0001 C CNN
