File: electrical/ECU/kicad_ECU/adc_clamp.sch (KiCad schematic (older format))
At the start: 1 part, among them U11 ESD7004

Commit message: minor naming change
Parts:
- renumbered U11 to U1401
Changed lines of the file:
@@
 $EndDescr
 $Comp
-L ESD7004 U11
+L ESD7004 U1401
 U 1 1 59774F90
 P 5950 3350
-F 0 "U11" H 5950 3250 50  0000 C CNN
+F 0 "U1401" H 5950 3250 50  0000 C CNN
 F 1 "ESD7004" H 5950 3450 50  0000 C CNN
 F 2 "MODULE" H 5950 3350 50  0001 C CNN
@@
 $EndComp
 $Comp
-L Earth #PWR052
+L Earth #PWR1402
 U 1 1 59774FB7
 P 7050 4100
-F 0 "#PWR052" H 7050 3850 50  0001 C CNN
+F 0 "#PWR1402" H 7050 3850 50  0001 C CNN
 F 1 "Earth" H 7050 3950 50  0001 C CNN
 F 2 "" H 7050 4100 50  0001 C CNN
@@
 $EndComp
 $Comp
-L Earth #PWR053
+L Earth #PWR1401
 U 1 1 59774FCD
 P 4350 4100
-F 0 "#PWR053" H 4350 3850 50  0001 C CNN
+F 0 "#PWR1401" H 4350 3850 50  0001 C CNN
 F 1 "Earth" H 4350 3950 50  0001 C CNN
 F 2 "" H 4350 4100 50  0001 C CNN
