File: electrical/ECU/kicad_ECU/airhead_ecu.sch (KiCad schematic (older format))
At the start: 6 parts, among them P1 CONN_01X04, P2 CONN_01X04, U1 10si_rect, U2 Mini50p16

Commit message: minor naming change
Parts:
- D101: renamed from 3A1; value D -> 3A
- D102: renamed from 3A2; value D -> 3A
- renumbered P1 to P101, P2 to P102, U1 to U101, U2 to U102
Changed lines of the file:
@@
 $EndDescr
 $Comp
-L D 3A1
+L D D101
 U 1 1 58897A54
 P 4400 5200
-F 0 "3A1" H 4400 5300 50  0000 C CNN
-F 1 "D" H 4400 5100 50  0000 C CNN
+F 0 "D101" H 4400 5300 50  0000 C CNN
+F 1 "3A" H 4400 5100 50  0000 C CNN
 F 2 "" H 4400 5200 50  0000 C CNN
 F 3 "" H 4400 5200 50  0000 C CNN
@@
 $EndComp
 $Comp
-L D 3A2
+L D D102
 U 1 1 58897A8D
 P 4700 5200
-F 0 "3A2" H 4700 5300 50  0000 C CNN
-F 1 "D" H 4700 5100 50  0000 C CNN
+F 0 "D102" H 4700 5300 50  0000 C CNN
+F 1 "3A" H 4700 5100 50  0000 C CNN
 F 2 "" H 4700 5200 50  0000 C CNN
 F 3 "" H 4700 5200 50  0000 C CNN
@@
 $EndComp
 $Comp
-L CONN_01X04 P1
+L CONN_01X04 P101
 U 1 1 58977F64
 P 1100 4800
-F 0 "P1" H 1100 5050 50  0000 C CNN
+F 0 "P101" H 1100 5050 50  0000 C CNN
 F 1 "CONN_01X04" V 1200 4800 50  0000 C CNN
 F 2 "" H 1100 4800 50  0000 C CNN
@@
 $EndComp
 $Comp
-L CONN_01X04 P2
+L CONN_01X04 P102
 U 1 1 58977F99
 P 1150 3250
-F 0 "P2" H 1150 3500 50  0000 C CNN
+F 0 "P102" H 1150 3500 50  0000 C CNN
 F 1 "CONN_01X04" V 1250 3250 50  0000 C CNN
 F 2 "" H 1150 3250 50  0000 C CNN
@@
 $EndComp
 $Comp
-L Earth #PWR01
+L Earth #PWR104
 U 1 1 5898F0D8
 P 4700 5650
-F 0 "#PWR01" H 4700 5400 50  0001 C CNN
+F 0 "#PWR104" H 4700 5400 50  0001 C CNN
 F 1 "Earth" H 4700 5500 50  0001 C CNN
 F 2 "" H 4700 5650 50  0000 C CNN
@@
 12v
 $Comp
-L 10si_rect U1
+L 10si_rect U101
 U 1 1 597E65C7
 P 1100 6650
-F 0 "U1" H 1100 6550 50  0000 C CNN
+F 0 "U101" H 1100 6550 50  0000 C CNN
 F 1 "10si_rect" H 1100 6750 50  0000 C CNN
 F 2 "MODULE" H 1100 6650 50  0001 C CNN
@@
 12v
 $Comp
-L PWR_FLAG #FLG02
+L PWR_FLAG #FLG103
 U 1 1 597E73C4
 P 2400 6650
-F 0 "#FLG02" H 2400 6725 50  0001 C CNN
+F 0 "#FLG103" H 2400 6725 50  0001 C CNN
 F 1 "PWR_FLAG" H 2400 6800 50  0000 C CNN
 F 2 "" H 2400 6650 50  0001 C CNN
@@
 $EndComp
 $Comp
-L Earth #PWR03
+L Earth #PWR102
 U 1 1 597E7602
 P 2750 7000
-F 0 "#PWR03" H 2750 6750 50  0001 C CNN
+F 0 "#PWR102" H 2750 6750 50  0001 C CNN
 F 1 "Earth" H 2750 6850 50  0001 C CNN
 F 2 "" H 2750 7000 50  0001 C CNN
@@
 Connection ~ 4550 4650
 $Comp
-L Mini50p16 U2
+L Mini50p16 U102
 U 1 1 59804CF3
 P 2250 1400
-F 0 "U2" H 2250 1400 50  0000 C CNN
+F 0 "U102" H 2250 1400 50  0000 C CNN
 F 1 "Mini50p16" H 2250 1600 50  0000 C CNN
 F 2 "MODULE" H 2250 1500 50  0001 C CNN
@@
 	750  1150 750  2100
 $Comp
-L Earth #PWR04
+L Earth #PWR101
 U 1 1 598074B3
 P 750 2100
-F 0 "#PWR04" H 750 1850 50  0001 C CNN
+F 0 "#PWR101" H 750 1850 50  0001 C CNN
 F 1 "Earth" H 750 1950 50  0001 C CNN
 F 2 "" H 750 2100 50  0001 C CNN
@@
 	3750 1250 3750 2200
 $Comp
-L Earth #PWR05
+L Earth #PWR103
 U 1 1 59807753
 P 3750 2200
-F 0 "#PWR05" H 3750 1950 50  0001 C CNN
+F 0 "#PWR103" H 3750 1950 50  0001 C CNN
 F 1 "Earth" H 3750 2050 50  0001 C CNN
 F 2 "" H 3750 2200 50  0001 C CNN
@@
 Connection ~ 2400 6650
 $Comp
-L PWR_FLAG #FLG06
+L PWR_FLAG #FLG102
 U 1 1 5990DA86
 P 1900 6750
-F 0 "#FLG06" H 1900 6825 50  0001 C CNN
+F 0 "#FLG102" H 1900 6825 50  0001 C CNN
 F 1 "PWR_FLAG" H 1900 6900 50  0000 C CNN
 F 2 "" H 1900 6750 50  0001 C CNN
@@
 Connection ~ 1900 6750
 $Comp
-L PWR_FLAG #FLG07
+L PWR_FLAG #FLG101
 U 1 1 5990DC10
 P 1450 950
-F 0 "#FLG07" H 1450 1025 50  0001 C CNN
+F 0 "#FLG101" H 1450 1025 50  0001 C CNN
 F 1 "PWR_FLAG" H 1450 1100 50  0000 C CNN
 F 2 "" H 1450 950 50  0001 C CNN
@@
 Connection ~ 1450 950
 $Comp
-L PWR_FLAG #FLG08
+L PWR_FLAG #FLG104
 U 1 1 5991C36F
 P 7050 1100
-F 0 "#FLG08" H 7050 1175 50  0001 C CNN
+F 0 "#FLG104" H 7050 1175 50  0001 C CNN
 F 1 "PWR_FLAG" H 7050 1250 50  0000 C CNN
 F 2 "" H 7050 1100 50  0001 C CNN
