File: electrical/ECU/kicad_ECU/antenna.sch (KiCad schematic (older format))
At the start: 4 parts

Commit message: minor naming change
Parts:
- renumbered AE1 to AE801, B1 to B801, L5 to L801, L6 to L802
Changed lines of the file:
@@
 $EndDescr
 $Comp
-L 2450BM14E0003 B1
+L 2450BM14E0003 B801
 U 1 1 59818520
 P 5750 3350
-AR Path="/597003E2/598181D1/59818520" Ref="B1"  Part="1"
-AR Path="/5978A36B/59800725/59818520" Ref="B2"  Part="1"
-F 0 "B2" H 5450 3750 60  0000 L CNN
+AR Path="/597003E2/598181D1/59818520" Ref="B801"  Part="1"
+AR Path="/5978A36B/59800725/59818520" Ref="B3201"  Part="1"
+F 0 "B3201" H 5450 3750 60  0000 L CNN
 F 1 "2450BM14E0003" H 5750 2950 60  0000 C CNN
 F 2 "" H 5750 3350 60  0000 C CNN
@@
 $EndComp
 $Comp
-L L L5
+L L L801
 U 1 1 59818535
 P 6750 3200
-AR Path="/597003E2/598181D1/59818535" Ref="L5"  Part="1"
-AR Path="/5978A36B/59800725/59818535" Ref="L8"  Part="1"
-F 0 "L8" V 6700 3200 50  0000 C CNN
+AR Path="/597003E2/598181D1/59818535" Ref="L801"  Part="1"
+AR Path="/5978A36B/59800725/59818535" Ref="L3201"  Part="1"
+F 0 "L3201" V 6700 3200 50  0000 C CNN
 F 1 "LQG15HH6N2S02D" V 6825 3200 50  0000 C CNN
 F 2 "" H 6750 3200 50  0001 C CNN
@@
 $EndComp
 $Comp
-L Antenna AE1
+L Antenna AE801
 U 1 1 5981853C
 P 7550 3000
-AR Path="/597003E2/598181D1/5981853C" Ref="AE1"  Part="1"
-AR Path="/5978A36B/59800725/5981853C" Ref="AE2"  Part="1"
-F 0 "AE2" H 7475 3075 50  0000 R CNN
+AR Path="/597003E2/598181D1/5981853C" Ref="AE801"  Part="1"
+AR Path="/5978A36B/59800725/5981853C" Ref="AE3201"  Part="1"
+F 0 "AE3201" H 7475 3075 50  0000 R CNN
 F 1 "146175" H 7475 3000 50  0000 R CNN
 F 2 "" H 7550 3000 50  0001 C CNN
@@
 $EndComp
 $Comp
-L L L6
+L L L802
 U 1 1 59818543
 P 7200 3650
-AR Path="/597003E2/598181D1/59818543" Ref="L6"  Part="1"
-AR Path="/5978A36B/59800725/59818543" Ref="L9"  Part="1"
-F 0 "L9" V 7150 3650 50  0000 C CNN
+AR Path="/597003E2/598181D1/59818543" Ref="L802"  Part="1"
+AR Path="/5978A36B/59800725/59818543" Ref="L3202"  Part="1"
+F 0 "L3202" V 7150 3650 50  0000 C CNN
 F 1 "LQG15HH5N6S02D" V 7275 3650 50  0000 C CNN
 F 2 "" H 7200 3650 50  0001 C CNN
@@
 $EndComp
 $Comp
-L Earth #PWR037
+L Earth #PWR801
 U 1 1 5981854A
 P 7200 4100
-AR Path="/597003E2/598181D1/5981854A" Ref="#PWR037"  Part="1"
-AR Path="/5978A36B/59800725/5981854A" Ref="#PWR082"  Part="1"
-F 0 "#PWR082" H 7200 3850 50  0001 C CNN
+AR Path="/597003E2/598181D1/5981854A" Ref="#PWR801"  Part="1"
+AR Path="/5978A36B/59800725/5981854A" Ref="#PWR3201"  Part="1"
+F 0 "#PWR3201" H 7200 3850 50  0001 C CNN
 F 1 "Earth" H 7200 3950 50  0001 C CNN
 F 2 "" H 7200 4100 50  0001 C CNN
