File: electrical/ECU/kicad_ECU/coil_driver.sch (KiCad schematic (older format))
At the start: 6 parts, among them U14 VB525SP-E

Commit message: minor naming change
Parts:
- renumbered C43 to C1901, C44 to C1902, C45 to C1903, R37 to R1901, R38 to R1902, U14 to U1901
Changed lines of the file:
@@
 $EndDescr
 $Comp
-L VB525SP-E U14
+L VB525SP-E U1901
 U 1 1 58AD2D12
 P 6500 3300
-AR Path="/5974D512/59776B36/58AD2D12" Ref="U14"  Part="1"
-AR Path="/5974D512/59776B4C/58AD2D12" Ref="U15"  Part="1"
-F 0 "U15" H 6550 3350 50  0000 C CNN
+AR Path="/5974D512/59776B36/58AD2D12" Ref="U1901"  Part="1"
+AR Path="/5974D512/59776B4C/58AD2D12" Ref="U2001"  Part="1"
+F 0 "U2001" H 6550 3350 50  0000 C CNN
 F 1 "VB525SP-E" H 6500 3400 50  0000 C CNN
 F 2 "MODULE" H 6500 3300 50  0001 C CNN
@@
 NoConn ~ 5700 3300
 $Comp
-L C_Small C44
+L C_Small C1902
 U 1 1 58AD2D1A
 P 5700 2500
-AR Path="/5974D512/59776B36/58AD2D1A" Ref="C44"  Part="1"
-AR Path="/5974D512/59776B4C/58AD2D1A" Ref="C47"  Part="1"
-F 0 "C47" H 5710 2570 50  0000 L CNN
+AR Path="/5974D512/59776B36/58AD2D1A" Ref="C1902"  Part="1"
+AR Path="/5974D512/59776B4C/58AD2D1A" Ref="C2002"  Part="1"
+F 0 "C2002" H 5710 2570 50  0000 L CNN
 F 1 "1uF" H 5710 2420 50  0000 L CNN
 F 2 "" H 5700 2500 50  0000 C CNN
@@
 $EndComp
 $Comp
-L C_Small C45
+L C_Small C1903
 U 1 1 58AD2D21
 P 5700 2750
-AR Path="/5974D512/59776B36/58AD2D21" Ref="C45"  Part="1"
-AR Path="/5974D512/59776B4C/58AD2D21" Ref="C48"  Part="1"
-F 0 "C48" H 5710 2820 50  0000 L CNN
+AR Path="/5974D512/59776B36/58AD2D21" Ref="C1903"  Part="1"
+AR Path="/5974D512/59776B4C/58AD2D21" Ref="C2003"  Part="1"
+F 0 "C2003" H 5710 2820 50  0000 L CNN
 F 1 "100nF" H 5710 2670 50  0000 L CNN
 F 2 "" H 5700 2750 50  0000 C CNN
@@
 $EndComp
 $Comp
-L R_Small R38
+L R_Small R1902
 U 1 1 58AD2D28
 P 5600 3500
-AR Path="/5974D512/59776B36/58AD2D28" Ref="R38"  Part="1"
-AR Path="/5974D512/59776B4C/58AD2D28" Ref="R40"  Part="1"
-F 0 "R40" H 5630 3520 50  0000 L CNN
+AR Path="/5974D512/59776B36/58AD2D28" Ref="R1902"  Part="1"
+AR Path="/5974D512/59776B4C/58AD2D28" Ref="R2002"  Part="1"
+F 0 "R2002" H 5630 3520 50  0000 L CNN
 F 1 "1k" H 5630 3460 50  0000 L CNN
 F 2 "" H 5600 3500 50  0000 C CNN
@@
 $EndComp
 $Comp
-L R_Small R37
+L R_Small R1901
 U 1 1 58AD2D2F
 P 5450 3750
-AR Path="/5974D512/59776B36/58AD2D2F" Ref="R37"  Part="1"
-AR Path="/5974D512/59776B4C/58AD2D2F" Ref="R39"  Part="1"
-F 0 "R39" H 5480 3770 50  0000 L CNN
+AR Path="/5974D512/59776B36/58AD2D2F" Ref="R1901"  Part="1"
+AR Path="/5974D512/59776B4C/58AD2D2F" Ref="R2001"  Part="1"
+F 0 "R2001" H 5480 3770 50  0000 L CNN
 F 1 "18k" H 5480 3710 50  0000 L CNN
 F 2 "" H 5450 3750 50  0000 C CNN
@@
 $EndComp
 $Comp
-L C_Small C43
+L C_Small C1901
 U 1 1 58AD2D36
 P 5150 3750
-AR Path="/5974D512/59776B36/58AD2D36" Ref="C43"  Part="1"
-AR Path="/5974D512/59776B4C/58AD2D36" Ref="C46"  Part="1"
-F 0 "C46" H 5160 3820 50  0000 L CNN
+AR Path="/5974D512/59776B36/58AD2D36" Ref="C1901"  Part="1"
+AR Path="/5974D512/59776B4C/58AD2D36" Ref="C2001"  Part="1"
+F 0 "C2001" H 5160 3820 50  0000 L CNN
 F 1 "1nF" H 5160 3670 50  0000 L CNN
 F 2 "" H 5150 3750 50  0000 C CNN
@@
 	7400 4300 7400 2750
 $Comp
-L Earth #PWR058
+L Earth #PWR1901
 U 1 1 599462B9
 P 6900 4550
-AR Path="/5974D512/59776B36/599462B9" Ref="#PWR058"  Part="1"
-AR Path="/5974D512/59776B4C/599462B9" Ref="#PWR059"  Part="1"
-F 0 "#PWR059" H 6900 4300 50  0001 C CNN
+AR Path="/5974D512/59776B36/599462B9" Ref="#PWR1901"  Part="1"
+AR Path="/5974D512/59776B4C/599462B9" Ref="#PWR2001"  Part="1"
+F 0 "#PWR2001" H 6900 4300 50  0001 C CNN
 F 1 "Earth" H 6900 4400 50  0001 C CNN
 F 2 "" H 6900 4550 50  0001 C CNN
