File: electrical/ECU/kicad_ECU/debug_leds.sch (KiCad schematic (older format))
At the start: 6 parts, among them SW3 SW_Push_Dual, SW4 SW_Push_Dual, SW5 SW_Push_Dual

Commit message: minor naming change
Parts:
- renumbered R72 to R2601, R73 to R2602, R74 to R2603, SW3 to SW2601, SW4 to SW2602, SW5 to SW2603
Changed lines of the file:
@@
 RCK
 $Comp
-L SW_Push_Dual SW3
+L SW_Push_Dual SW2601
 U 1 1 597CD809
 P 3300 4400
-F 0 "SW3" H 3350 4500 50  0000 L CNN
+F 0 "SW2601" H 3350 4500 50  0000 L CNN
 F 1 "SW_Push_Dual" H 3300 4130 50  0000 C CNN
 F 2 "" H 3300 4600 50  0001 C CNN
@@
 Connection ~ 3700 4400
 $Comp
-L R R72
+L R R2601
 U 1 1 597CE2D4
 P 4150 4700
-F 0 "R72" V 4230 4700 50  0000 C CNN
+F 0 "R2601" V 4230 4700 50  0000 C CNN
 F 1 "10k" V 4150 4700 50  0000 C CNN
 F 2 "" V 4080 4700 50  0001 C CNN
@@
 	4150 4850 4150 5100
 $Comp
-L SW_Push_Dual SW4
+L SW_Push_Dual SW2602
 U 1 1 597CE671
 P 6250 4400
-F 0 "SW4" H 6300 4500 50  0000 L CNN
+F 0 "SW2602" H 6300 4500 50  0000 L CNN
 F 1 "SW_Push_Dual" H 6250 4130 50  0000 C CNN
 F 2 "" H 6250 4600 50  0001 C CNN
@@
 Connection ~ 6650 4400
 $Comp
-L R R73
+L R R2602
 U 1 1 597CE681
 P 7100 4700
-F 0 "R73" V 7180 4700 50  0000 C CNN
+F 0 "R2602" V 7180 4700 50  0000 C CNN
 F 1 "10k" V 7100 4700 50  0000 C CNN
 F 2 "" V 7030 4700 50  0001 C CNN
@@
 	7100 4850 7100 5550
 $Comp
-L SW_Push_Dual SW5
+L SW_Push_Dual SW2603
 U 1 1 597CE819
 P 9100 4400
-F 0 "SW5" H 9150 4500 50  0000 L CNN
+F 0 "SW2603" H 9150 4500 50  0000 L CNN
 F 1 "SW_Push_Dual" H 9100 4130 50  0000 C CNN
 F 2 "" H 9100 4600 50  0001 C CNN
@@
 Connection ~ 9500 4400
 $Comp
-L R R74
+L R R2603
 U 1 1 597CE829
 P 9950 4700
-F 0 "R74" V 10030 4700 50  0000 C CNN
+F 0 "R2603" V 10030 4700 50  0000 C CNN
 F 1 "10k" V 9950 4700 50  0000 C CNN
 F 2 "" V 9880 4700 50  0001 C CNN
@@
 	9950 5100 9950 4850
 $Comp
-L Earth #PWR078
+L Earth #PWR2601
 U 1 1 59922A45
 P 7100 5550
-F 0 "#PWR078" H 7100 5300 50  0001 C CNN
+F 0 "#PWR2601" H 7100 5300 50  0001 C CNN
 F 1 "Earth" H 7100 5400 50  0001 C CNN
 F 2 "" H 7100 5550 50  0001 C CNN
