File: electrical/ECU/kicad_ECU/ext_protection.sch (KiCad schematic (older format))
At the start: 8 parts

Commit message: minor naming change
Parts:
- renumbered D_Zener2 to D_Zener3101, D_Zener3 to D_Zener3102, D_Zener4 to D_Zener3103, D_Zener5 to D_Zener3104, Polyfuse1 to Polyfuse3101, Polyfuse2 to Polyfuse3102, Polyfuse3 to Polyfuse3103, Polyfuse4 to Polyfuse3104
Changed lines of the file:
@@
 OUT1
 $Comp
-L Polyfuse Polyfuse1
+L Polyfuse Polyfuse3101
 U 1 1 597FE5B1
 P 6400 2550
-F 0 "Polyfuse1" V 6300 2550 50  0000 C CNN
+F 0 "Polyfuse3101" V 6300 2550 50  0000 C CNN
 F 1 "30mA" V 6500 2550 50  0000 C CNN
 F 2 "" H 6450 2350 50  0001 L CNN
@@
 	4850 2550 6250 2550
 $Comp
-L D_Zener D_Zener2
+L D_Zener D_Zener3101
 U 1 1 597FE5BA
 P 5200 3900
-F 0 "D_Zener2" H 5200 4000 50  0000 C CNN
+F 0 "D_Zener3101" H 5200 4000 50  0000 C CNN
 F 1 "3.38v" H 5200 3800 50  0000 C CNN
 F 2 "" H 5200 3900 50  0001 C CNN
@@
 	4850 3150 6250 3150
 $Comp
-L Earth #PWR081
+L Earth #PWR3101
 U 1 1 597FE5E9
 P 5650 4350
-F 0 "#PWR081" H 5650 4100 50  0001 C CNN
+F 0 "#PWR3101" H 5650 4100 50  0001 C CNN
 F 1 "Earth" H 5650 4200 50  0001 C CNN
 F 2 "" H 5650 4350 50  0001 C CNN
@@
 PIN4
 $Comp
-L Polyfuse Polyfuse2
+L Polyfuse Polyfuse3102
 U 1 1 59961BEE
 P 6400 2850
-F 0 "Polyfuse2" V 6300 2850 50  0000 C CNN
+F 0 "Polyfuse3102" V 6300 2850 50  0000 C CNN
 F 1 "30mA" V 6500 2850 50  0000 C CNN
 F 2 "" H 6450 2650 50  0001 L CNN
@@
 $EndComp
 $Comp
-L Polyfuse Polyfuse3
+L Polyfuse Polyfuse3103
 U 1 1 59961C1E
 P 6400 3150
-F 0 "Polyfuse3" V 6300 3150 50  0000 C CNN
+F 0 "Polyfuse3103" V 6300 3150 50  0000 C CNN
 F 1 "30mA" V 6500 3150 50  0000 C CNN
 F 2 "" H 6450 2950 50  0001 L CNN
@@
 $EndComp
 $Comp
-L Polyfuse Polyfuse4
+L Polyfuse Polyfuse3104
 U 1 1 59961C53
 P 6400 3450
-F 0 "Polyfuse4" V 6300 3450 50  0000 C CNN
+F 0 "Polyfuse3104" V 6300 3450 50  0000 C CNN
 F 1 "30mA" V 6500 3450 50  0000 C CNN
 F 2 "" H 6450 3250 50  0001 L CNN
@@
 $EndComp
 $Comp
-L D_Zener D_Zener3
+L D_Zener D_Zener3102
 U 1 1 59961CCE
 P 5500 3900
-F 0 "D_Zener3" H 5500 4000 50  0000 C CNN
+F 0 "D_Zener3102" H 5500 4000 50  0000 C CNN
 F 1 "3.38v" H 5500 3800 50  0000 C CNN
 F 2 "" H 5500 3900 50  0001 C CNN
@@
 $EndComp
 $Comp
-L D_Zener D_Zener4
+L D_Zener D_Zener3103
 U 1 1 59961CF9
 P 5800 3900
-F 0 "D_Zener4" H 5800 4000 50  0000 C CNN
+F 0 "D_Zener3103" H 5800 4000 50  0000 C CNN
 F 1 "3.38v" H 5800 3800 50  0000 C CNN
 F 2 "" H 5800 3900 50  0001 C CNN
@@
 $EndComp
 $Comp
-L D_Zener D_Zener5
+L D_Zener D_Zener3104
 U 1 1 59961D22
 P 6100 3900
-F 0 "D_Zener5" H 6100 4000 50  0000 C CNN
+F 0 "D_Zener3104" H 6100 4000 50  0000 C CNN
 F 1 "3.38v" H 6100 3800 50  0000 C CNN
 F 2 "" H 6100 3900 50  0001 C CNN
