File: electrical/ECU/kicad_ECU/high_current.sch (KiCad schematic (older format))
At the start: 5 parts, among them U16 BSC072N03LD-G

Commit message: minor naming change
Parts:
- renumbered R41 to R2101, R42 to R2102, R43 to R2103, R44 to R2104, U16 to U2101
Changed lines of the file:
@@
 $EndDescr
 $Comp
-L BSC072N03LD-G U16
+L BSC072N03LD-G U2101
 U 1 1 5977C2D7
 P 6600 3150
-F 0 "U16" H 6600 3050 50  0000 C CNN
+F 0 "U2101" H 6600 3050 50  0000 C CNN
 F 1 "BSC072N03LD-G" H 6600 3250 50  0000 C CNN
 F 2 "MODULE" H 6600 3150 50  0001 C CNN
@@
 $EndComp
 $Comp
-L R R43
+L R R2103
 U 1 1 5977C2E4
 P 5200 3100
-F 0 "R43" V 5280 3100 50  0000 C CNN
+F 0 "R2103" V 5280 3100 50  0000 C CNN
 F 1 "1k" V 5200 3100 50  0000 C CNN
 F 2 "" V 5130 3100 50  0001 C CNN
@@
 $EndComp
 $Comp
-L R R44
+L R R2104
 U 1 1 5977C2EB
 P 5200 3300
-F 0 "R44" V 5280 3300 50  0000 C CNN
+F 0 "R2104" V 5280 3300 50  0000 C CNN
 F 1 "1k" V 5200 3300 50  0000 C CNN
 F 2 "" V 5130 3300 50  0001 C CNN
@@
 $EndComp
 $Comp
-L R R42
+L R R2102
 U 1 1 5977C2F2
 P 4850 3600
-F 0 "R42" V 4930 3600 50  0000 C CNN
+F 0 "R2102" V 4930 3600 50  0000 C CNN
 F 1 "100k" V 4850 3600 50  0000 C CNN
 F 2 "" V 4780 3600 50  0001 C CNN
@@
 $EndComp
 $Comp
-L R R41
+L R R2101
 U 1 1 5977C2F9
 P 4600 3600
-F 0 "R41" V 4680 3600 50  0000 C CNN
+F 0 "R2101" V 4680 3600 50  0000 C CNN
 F 1 "100k" V 4600 3600 50  0000 C CNN
 F 2 "" V 4530 3600 50  0001 C CNN
@@
 	7550 3200 7550 3300
 $Comp
-L Earth #PWR060
+L Earth #PWR2101
 U 1 1 599401D9
 P 4600 4150
-F 0 "#PWR060" H 4600 3900 50  0001 C CNN
+F 0 "#PWR2101" H 4600 3900 50  0001 C CNN
 F 1 "Earth" H 4600 4000 50  0001 C CNN
 F 2 "" H 4600 4150 50  0001 C CNN
@@
 $EndComp
 $Comp
-L Earth #PWR061
+L Earth #PWR2102
 U 1 1 599401F7
 P 5600 4150
-F 0 "#PWR061" H 5600 3900 50  0001 C CNN
+F 0 "#PWR2102" H 5600 3900 50  0001 C CNN
 F 1 "Earth" H 5600 4000 50  0001 C CNN
 F 2 "" H 5600 4150 50  0001 C CNN
