File: electrical/ECU/kicad_ECU/injectors.sch (KiCad schematic (older format))
At the start: 11 parts, among them U17 BSC072N03LD-G

Commit message: minor naming change
Parts:
- renumbered D31 to D2201, D32 to D2202, D33 to D2203, D34 to D2204, R45 to R2201, R46 to R2202, R47 to R2203, R48 to R2204, R49 to R2205, R50 to R2206, U17 to U2201
Changed lines of the file:
@@
 $EndDescr
 $Comp
-L BSC072N03LD-G U17
+L BSC072N03LD-G U2201
 U 1 1 5977A542
 P 7250 3250
-F 0 "U17" H 7250 3150 50  0000 C CNN
+F 0 "U2201" H 7250 3150 50  0000 C CNN
 F 1 "BSC072N03LD-G" H 7250 3350 50  0000 C CNN
 F 2 "MODULE" H 7250 3250 50  0001 C CNN
@@
 $EndComp
 $Comp
-L Earth #PWR062
+L Earth #PWR2201
 U 1 1 5977A637
 P 6250 4100
-F 0 "#PWR062" H 6250 3850 50  0001 C CNN
+F 0 "#PWR2201" H 6250 3850 50  0001 C CNN
 F 1 "Earth" H 6250 3950 50  0001 C CNN
 F 2 "" H 6250 4100 50  0001 C CNN
@@
 $EndComp
 $Comp
-L R R47
+L R R2203
 U 1 1 5977A67E
 P 5850 3200
-F 0 "R47" V 5930 3200 50  0000 C CNN
+F 0 "R2203" V 5930 3200 50  0000 C CNN
 F 1 "1k" V 5850 3200 50  0000 C CNN
 F 2 "" V 5780 3200 50  0001 C CNN
@@
 $EndComp
 $Comp
-L R R48
+L R R2204
 U 1 1 5977A6ED
 P 5850 3400
-F 0 "R48" V 5930 3400 50  0000 C CNN
+F 0 "R2204" V 5930 3400 50  0000 C CNN
 F 1 "1k" V 5850 3400 50  0000 C CNN
 F 2 "" V 5780 3400 50  0001 C CNN
@@
 $EndComp
 $Comp
-L R R46
+L R R2202
 U 1 1 5977A71B
 P 5500 3700
-F 0 "R46" V 5580 3700 50  0000 C CNN
+F 0 "R2202" V 5580 3700 50  0000 C CNN
 F 1 "100k" V 5500 3700 50  0000 C CNN
 F 2 "" V 5430 3700 50  0001 C CNN
@@
 $EndComp
 $Comp
-L R R45
+L R R2201
 U 1 1 5977A73E
 P 5250 3700
-F 0 "R45" V 5330 3700 50  0000 C CNN
+F 0 "R2201" V 5330 3700 50  0000 C CNN
 F 1 "100k" V 5250 3700 50  0000 C CNN
 F 2 "" V 5180 3700 50  0001 C CNN
@@
 INJ2-CPU
 $Comp
-L D D33
+L D D2203
 U 1 1 5977A82B
 P 7700 2600
-F 0 "D33" H 7700 2700 50  0000 C CNN
+F 0 "D2203" H 7700 2700 50  0000 C CNN
 F 1 "1N4004" H 7700 2500 50  0000 C CNN
 F 2 "" H 7700 2600 50  0001 C CNN
@@
 $EndComp
 $Comp
-L LED-RESCUE-airhead_ecu D31
+L LED-RESCUE-airhead_ecu D2201
 U 1 1 5977A89D
 P 6900 2600
-F 0 "D31" H 6900 2700 50  0000 C CNN
+F 0 "D2201" H 6900 2700 50  0000 C CNN
 F 1 "LED" H 6900 2500 50  0000 C CNN
 F 2 "" H 6900 2600 50  0001 C CNN
@@
 $EndComp
 $Comp
-L R R49
+L R R2205
 U 1 1 5977A8EA
 P 6050 2600
-F 0 "R49" V 6130 2600 50  0000 C CNN
+F 0 "R2205" V 6130 2600 50  0000 C CNN
 F 1 "680" V 6050 2600 50  0000 C CNN
 F 2 "" V 5980 2600 50  0001 C CNN
@@
 12v
 $Comp
-L D D34
+L D D2204
 U 1 1 5977AA87
 P 7700 4550
-F 0 "D34" H 7700 4650 50  0000 C CNN
+F 0 "D2204" H 7700 4650 50  0000 C CNN
 F 1 "1N4004" H 7700 4450 50  0000 C CNN
 F 2 "" H 7700 4550 50  0001 C CNN
@@
 $EndComp
 $Comp
-L LED-RESCUE-airhead_ecu D32
+L LED-RESCUE-airhead_ecu D2202
 U 1 1 5977AA8D
 P 6900 4550
-F 0 "D32" H 6900 4650 50  0000 C CNN
+F 0 "D2202" H 6900 4650 50  0000 C CNN
 F 1 "LED" H 6900 4450 50  0000 C CNN
 F 2 "" H 6900 4550 50  0001 C CNN
@@
 $EndComp
 $Comp
-L R R50
+L R R2206
 U 1 1 5977AA93
 P 6050 4550
-F 0 "R50" V 6130 4550 50  0000 C CNN
+F 0 "R2206" V 6130 4550 50  0000 C CNN
 F 1 "680" V 6050 4550 50  0000 C CNN
 F 2 "" V 5980 4550 50  0001 C CNN
