File: electrical/ECU/kicad_ECU/level_shifter.sch (KiCad schematic (older format))
At the start: 24 parts, among them U20 NTB0101AGWH, U21 NTB0101AGWH, U22 LMV822IQ2T, U23 LMV822IQ2T, U24 LMV822IQ2T

Commit message: minor naming change
Parts:
- renumbered C64 to C2501, C65 to C2502, C66 to C2503, C67 to C2504, C68 to C2505, C69 to C2506, C70 to C2507, R60 to R2501, R61 to R2502, R62 to R2503, R63 to R2504, R64 to R2505, R65 to R2506, R66 to R2507, R67 to R2508, R68 to R2509, R69 to R2510, R70 to R2511, R71 to R2512, U20 to U2501, U21 to U2502, U22 to U2503, U23 to U2504, U24 to U2505
Changed lines of the file:
@@
 coil2_5v_out
 $Comp
-L LMV822IQ2T U23
+L LMV822IQ2T U2504
 U 1 1 597915F5
 P 8500 1700
-F 0 "U23" H 8500 1600 50  0000 C CNN
+F 0 "U2504" H 8500 1600 50  0000 C CNN
 F 1 "LMV822IQ2T" H 8500 1800 50  0000 C CNN
 F 2 "MODULE" H 8500 1700 50  0001 C CNN
@@
 $EndComp
 $Comp
-L Earth #PWR071
+L Earth #PWR2506
 U 1 1 597916F8
 P 8500 2550
-F 0 "#PWR071" H 8500 2300 50  0001 C CNN
+F 0 "#PWR2506" H 8500 2300 50  0001 C CNN
 F 1 "Earth" H 8500 2400 50  0001 C CNN
 F 2 "" H 8500 2550 50  0001 C CNN
@@
 $EndComp
 $Comp
-L R R64
+L R R2505
 U 1 1 59791774
 P 6750 1500
-F 0 "R64" V 6830 1500 50  0000 C CNN
+F 0 "R2505" V 6830 1500 50  0000 C CNN
 F 1 "17k" V 6750 1500 50  0000 C CNN
 F 2 "" V 6680 1500 50  0001 C CNN
@@
 $EndComp
 $Comp
-L R R65
+L R R2506
 U 1 1 5979178D
 P 6750 2050
-F 0 "R65" V 6830 2050 50  0000 C CNN
+F 0 "R2506" V 6830 2050 50  0000 C CNN
 F 1 "33k" V 6750 2050 50  0000 C CNN
 F 2 "" V 6680 2050 50  0001 C CNN
@@
 $EndComp
 $Comp
-L C C69
+L C C2506
 U 1 1 597917D3
 P 9250 1200
-F 0 "C69" H 9275 1300 50  0000 L CNN
+F 0 "C2506" H 9275 1300 50  0000 L CNN
 F 1 "100nF" H 9275 1100 50  0000 L CNN
 F 2 "" H 9288 1050 50  0001 C CNN
@@
 Connection ~ 7750 2450
 $Comp
-L R R68
+L R R2509
 U 1 1 59791914
 P 10250 1600
-F 0 "R68" V 10330 1600 50  0000 C CNN
+F 0 "R2509" V 10330 1600 50  0000 C CNN
 F 1 "17k" V 10250 1600 50  0000 C CNN
 F 2 "" V 10180 1600 50  0001 C CNN
@@
 $EndComp
 $Comp
-L R R69
+L R R2510
 U 1 1 5979191A
 P 10250 2150
-F 0 "R69" V 10330 2150 50  0000 C CNN
+F 0 "R2510" V 10330 2150 50  0000 C CNN
 F 1 "33k" V 10250 2150 50  0000 C CNN
 F 2 "" V 10180 2150 50  0001 C CNN
@@
 MAP2_3v_out
 $Comp
-L LMV822IQ2T U24
+L LMV822IQ2T U2505
 U 1 1 59791C46
 P 8550 4500
-F 0 "U24" H 8550 4400 50  0000 C CNN
+F 0 "U2505" H 8550 4400 50  0000 C CNN
 F 1 "LMV822IQ2T" H 8550 4600 50  0000 C CNN
 F 2 "MODULE" H 8550 4500 50  0001 C CNN
@@
 $EndComp
 $Comp
-L Earth #PWR072
+L Earth #PWR2507
 U 1 1 59791C4C
 P 8550 5350
-F 0 "#PWR072" H 8550 5100 50  0001 C CNN
+F 0 "#PWR2507" H 8550 5100 50  0001 C CNN
 F 1 "Earth" H 8550 5200 50  0001 C CNN
 F 2 "" H 8550 5350 50  0001 C CNN
@@
 $EndComp
 $Comp
-L R R66
+L R R2507
 U 1 1 59791C52
 P 6800 4300
-F 0 "R66" V 6880 4300 50  0000 C CNN
+F 0 "R2507" V 6880 4300 50  0000 C CNN
 F 1 "17k" V 6800 4300 50  0000 C CNN
 F 2 "" V 6730 4300 50  0001 C CNN
@@
 $EndComp
 $Comp
-L R R67
+L R R2508
 U 1 1 59791C58
 P 6800 4850
-F 0 "R67" V 6880 4850 50  0000 C CNN
+F 0 "R2508" V 6880 4850 50  0000 C CNN
 F 1 "33k" V 6800 4850 50  0000 C CNN
 F 2 "" V 6730 4850 50  0001 C CNN
@@
 $EndComp
 $Comp
-L C C70
+L C C2507
 U 1 1 59791C5E
 P 9300 4000
-F 0 "C70" H 9325 4100 50  0000 L CNN
+F 0 "C2507" H 9325 4100 50  0000 L CNN
 F 1 "100nF" H 9325 3900 50  0000 L CNN
 F 2 "" H 9338 3850 50  0001 C CNN
@@
 Connection ~ 7800 5250
 $Comp
-L R R70
+L R R2511
 U 1 1 59791C79
 P 10300 4400
-F 0 "R70" V 10380 4400 50  0000 C CNN
+F 0 "R2511" V 10380 4400 50  0000 C CNN
 F 1 "17k" V 10300 4400 50  0000 C CNN
 F 2 "" V 10230 4400 50  0001 C CNN
@@
 $EndComp
 $Comp
-L R R71
+L R R2512
 U 1 1 59791C7F
 P 10300 4950
-F 0 "R71" V 10380 4950 50  0000 C CNN
+F 0 "R2512" V 10380 4950 50  0000 C CNN
 F 1 "33k" V 10300 4950 50  0000 C CNN
 F 2 "" V 10230 4950 50  0001 C CNN
@@
 BRV_3v_out
 $Comp
-L LMV822IQ2T U22
+L LMV822IQ2T U2503
 U 1 1 59791E5C
 P 3500 6500
-F 0 "U22" H 3500 6400 50  0000 C CNN
+F 0 "U2503" H 3500 6400 50  0000 C CNN
 F 1 "LMV822IQ2T" H 3500 6600 50  0000 C CNN
 F 2 "MODULE" H 3500 6500 50  0001 C CNN
@@
 $EndComp
 $Comp
-L Earth #PWR073
+L Earth #PWR2503
 U 1 1 59791E62
 P 3500 7350
-F 0 "#PWR073" H 3500 7100 50  0001 C CNN
+F 0 "#PWR2503" H 3500 7100 50  0001 C CNN
 F 1 "Earth" H 3500 7200 50  0001 C CNN
 F 2 "" H 3500 7350 50  0001 C CNN
@@
 $EndComp
 $Comp
-L R R60
+L R R2501
 U 1 1 59791E68
 P 1750 6300
-F 0 "R60" V 1830 6300 50  0000 C CNN
+F 0 "R2501" V 1830 6300 50  0000 C CNN
 F 1 "17k" V 1750 6300 50  0000 C CNN
 F 2 "" V 1680 6300 50  0001 C CNN
@@
 $EndComp
 $Comp
-L R R61
+L R R2502
 U 1 1 59791E6E
 P 1750 6850
-F 0 "R61" V 1830 6850 50  0000 C CNN
+F 0 "R2502" V 1830 6850 50  0000 C CNN
 F 1 "33k" V 1750 6850 50  0000 C CNN
 F 2 "" V 1680 6850 50  0001 C CNN
@@
 $EndComp
 $Comp
-L C C66
+L C C2503
 U 1 1 59791E74
 P 4250 6000
-F 0 "C66" H 4275 6100 50  0000 L CNN
+F 0 "C2503" H 4275 6100 50  0000 L CNN
 F 1 "100nF" H 4275 5900 50  0000 L CNN
 F 2 "" H 4288 5850 50  0001 C CNN
@@
 Connection ~ 2750 7250
 $Comp
-L R R62
+L R R2503
 U 1 1 59791E8F
 P 5250 6400
-F 0 "R62" V 5330 6400 50  0000 C CNN
+F 0 "R2503" V 5330 6400 50  0000 C CNN
 F 1 "17k" V 5250 6400 50  0000 C CNN
 F 2 "" V 5180 6400 50  0001 C CNN
@@
 $EndComp
 $Comp
-L R R63
+L R R2504
 U 1 1 59791E95
 P 5250 6950
-F 0 "R63" V 5330 6950 50  0000 C CNN
+F 0 "R2504" V 5330 6950 50  0000 C CNN
 F 1 "33k" V 5250 6950 50  0000 C CNN
 F 2 "" V 5180 6950 50  0001 C CNN
@@
 Connection ~ 4400 6450
 $Comp
-L NTB0101AGWH U20
+L NTB0101AGWH U2501
 U 1 1 5979207E
 P 3400 1300
-F 0 "U20" H 3400 1200 50  0000 C CNN
+F 0 "U2501" H 3400 1200 50  0000 C CNN
 F 1 "NTB0101AGWH" H 3400 1400 50  0000 C CNN
 F 2 "MODULE" H 3400 1300 50  0001 C CNN
@@
 $EndComp
 $Comp
-L C C64
+L C C2501
 U 1 1 59792109
 P 2250 1700
-F 0 "C64" H 2275 1800 50  0000 L CNN
+F 0 "C2501" H 2275 1800 50  0000 L CNN
 F 1 "0.1uF" H 2275 1600 50  0000 L CNN
 F 2 "" H 2288 1550 50  0001 C CNN
@@
 $EndComp
 $Comp
-L Earth #PWR074
+L Earth #PWR2501
 U 1 1 5979219D
 P 2250 2150
-F 0 "#PWR074" H 2250 1900 50  0001 C CNN
+F 0 "#PWR2501" H 2250 1900 50  0001 C CNN
 F 1 "Earth" H 2250 2000 50  0001 C CNN
 F 2 "" H 2250 2150 50  0001 C CNN
@@
 Connection ~ 2250 2000
 $Comp
-L C C67
+L C C2504
 U 1 1 597926F6
 P 4550 1700
-F 0 "C67" H 4575 1800 50  0000 L CNN
+F 0 "C2504" H 4575 1800 50  0000 L CNN
 F 1 "0.1uF" H 4575 1600 50  0000 L CNN
 F 2 "" H 4588 1550 50  0001 C CNN
@@
 $EndComp
 $Comp
-L Earth #PWR075
+L Earth #PWR2504
 U 1 1 597926FC
 P 4550 2150
-F 0 "#PWR075" H 4550 1900 50  0001 C CNN
+F 0 "#PWR2504" H 4550 1900 50  0001 C CNN
 F 1 "Earth" H 4550 2000 50  0001 C CNN
 F 2 "" H 4550 2150 50  0001 C CNN
@@
 Connection ~ 4550 2000
 $Comp
-L NTB0101AGWH U21
+L NTB0101AGWH U2502
 U 1 1 597928D1
 P 3400 3550
-F 0 "U21" H 3400 3450 50  0000 C CNN
+F 0 "U2502" H 3400 3450 50  0000 C CNN
 F 1 "NTB0101AGWH" H 3400 3650 50  0000 C CNN
 F 2 "MODULE" H 3400 3550 50  0001 C CNN
@@
 $EndComp
 $Comp
-L C C65
+L C C2502
 U 1 1 597928D7
 P 2250 3950
-F 0 "C65" H 2275 4050 50  0000 L CNN
+F 0 "C2502" H 2275 4050 50  0000 L CNN
 F 1 "0.1uF" H 2275 3850 50  0000 L CNN
 F 2 "" H 2288 3800 50  0001 C CNN
@@
 $EndComp
 $Comp
-L Earth #PWR076
+L Earth #PWR2502
 U 1 1 597928DD
 P 2250 4400
-F 0 "#PWR076" H 2250 4150 50  0001 C CNN
+F 0 "#PWR2502" H 2250 4150 50  0001 C CNN
 F 1 "Earth" H 2250 4250 50  0001 C CNN
 F 2 "" H 2250 4400 50  0001 C CNN
@@
 Connection ~ 2250 4250
 $Comp
-L C C68
+L C C2505
 U 1 1 597928ED
 P 4550 3950
-F 0 "C68" H 4575 4050 50  0000 L CNN
+F 0 "C2505" H 4575 4050 50  0000 L CNN
 F 1 "0.1uF" H 4575 3850 50  0000 L CNN
 F 2 "" H 4588 3800 50  0001 C CNN
@@
 $EndComp
 $Comp
-L Earth #PWR077
+L Earth #PWR2505
 U 1 1 597928F3
 P 4550 4400
-F 0 "#PWR077" H 4550 4150 50  0001 C CNN
+F 0 "#PWR2505" H 4550 4150 50  0001 C CNN
 F 1 "Earth" H 4550 4250 50  0001 C CNN
 F 2 "" H 4550 4400 50  0001 C CNN
