File: electrical/ECU/kicad_ECU/map_subsystem.sch (KiCad schematic (older format))
At the start: 5 parts, among them U12 MPXA4250AC6U

Commit message: minor naming change
Parts:
- renumbered C37 to C1701, C38 to C1702, C39 to C1703, R35 to R1701, U12 to U1701
Changed lines of the file:
@@
 $EndDescr
 $Comp
-L MPXA4250AC6U U12
+L MPXA4250AC6U U1701
 U 1 1 5921F130
 P 6150 3100
-AR Path="/5974D512/59776310/5921F130" Ref="U12"  Part="1"
-AR Path="/5974D512/5977631A/5921F130" Ref="U13"  Part="1"
-F 0 "U13" H 6150 3000 50  0000 C CNN
+AR Path="/5974D512/59776310/5921F130" Ref="U1701"  Part="1"
+AR Path="/5974D512/5977631A/5921F130" Ref="U1801"  Part="1"
+F 0 "U1801" H 6150 3000 50  0000 C CNN
 F 1 "MPXA4250AC6U" H 6150 3200 50  0000 C CNN
 F 2 "MODULE" H 6150 3100 50  0001 C CNN
@@
 5vdc
 $Comp
-L Earth #PWR056
+L Earth #PWR1701
 U 1 1 5929DA6E
 P 4250 4200
-AR Path="/5974D512/59776310/5929DA6E" Ref="#PWR056"  Part="1"
-AR Path="/5974D512/5977631A/5929DA6E" Ref="#PWR057"  Part="1"
-F 0 "#PWR057" H 4250 3950 50  0001 C CNN
+AR Path="/5974D512/59776310/5929DA6E" Ref="#PWR1701"  Part="1"
+AR Path="/5974D512/5977631A/5929DA6E" Ref="#PWR1801"  Part="1"
+F 0 "#PWR1801" H 4250 3950 50  0001 C CNN
 F 1 "Earth" H 4250 4050 50  0001 C CNN
 F 2 "" H 4250 4200 50  0001 C CNN
@@
 PressA
 $Comp
-L R R35
+L R R1701
 U 1 1 5929DB00
 P 5100 3250
-AR Path="/5974D512/59776310/5929DB00" Ref="R35"  Part="1"
-AR Path="/5974D512/5977631A/5929DB00" Ref="R36"  Part="1"
-F 0 "R36" V 5180 3250 50  0000 C CNN
+AR Path="/5974D512/59776310/5929DB00" Ref="R1701"  Part="1"
+AR Path="/5974D512/5977631A/5929DB00" Ref="R1801"  Part="1"
+F 0 "R1801" V 5180 3250 50  0000 C CNN
 F 1 "470Ω" V 5100 3250 50  0000 C CNN
 F 2 "" V 5030 3250 50  0001 C CNN
@@
 	3500 3050 5400 3050
 $Comp
-L C C39
+L C C1703
 U 1 1 5929DF2C
 P 4600 3600
-AR Path="/5974D512/59776310/5929DF2C" Ref="C39"  Part="1"
-AR Path="/5974D512/5977631A/5929DF2C" Ref="C42"  Part="1"
-F 0 "C42" H 4625 3700 50  0000 L CNN
+AR Path="/5974D512/59776310/5929DF2C" Ref="C1703"  Part="1"
+AR Path="/5974D512/5977631A/5929DF2C" Ref="C1803"  Part="1"
+F 0 "C1803" H 4625 3700 50  0000 L CNN
 F 1 "0.3μF" H 4625 3500 50  0000 L CNN
 F 2 "" H 4638 3450 50  0001 C CNN
@@
 Connection ~ 4600 3250
 $Comp
-L C C38
+L C C1702
 U 1 1 5929DFD9
 P 4050 3600
-AR Path="/5974D512/59776310/5929DFD9" Ref="C38"  Part="1"
-AR Path="/5974D512/5977631A/5929DFD9" Ref="C41"  Part="1"
-F 0 "C41" H 4075 3700 50  0000 L CNN
+AR Path="/5974D512/59776310/5929DFD9" Ref="C1702"  Part="1"
+AR Path="/5974D512/5977631A/5929DFD9" Ref="C1802"  Part="1"
+F 0 "C1802" H 4075 3700 50  0000 L CNN
 F 1 "0.01μF" H 4075 3500 50  0000 L CNN
 F 2 "" H 4088 3450 50  0001 C CNN
@@
 $EndComp
 $Comp
-L C C37
+L C C1701
 U 1 1 5929DFF8
 P 3700 3600
-AR Path="/5974D512/59776310/5929DFF8" Ref="C37"  Part="1"
-AR Path="/5974D512/5977631A/5929DFF8" Ref="C40"  Part="1"
-F 0 "C40" H 3725 3700 50  0000 L CNN
+AR Path="/5974D512/59776310/5929DFF8" Ref="C1701"  Part="1"
+AR Path="/5974D512/5977631A/5929DFF8" Ref="C1801"  Part="1"
+F 0 "C1801" H 3725 3700 50  0000 L CNN
 F 1 "1μF" H 3725 3500 50  0000 L CNN
 F 2 "" H 3738 3450 50  0001 C CNN
