File: electrical/ECU/kicad_ECU/o2.sch (KiCad schematic (older format))
At the start: 3 parts

Commit message: minor naming change
Parts:
- renumbered C31 to C1301, C32 to C1302, R32 to R1301
Changed lines of the file:
@@
 CPU
 $Comp
-L R R32
+L R R1301
 U 1 1 597752E7
 P 5600 3250
-F 0 "R32" V 5680 3250 50  0000 C CNN
+F 0 "R1301" V 5680 3250 50  0000 C CNN
 F 1 "470" V 5600 3250 50  0000 C CNN
 F 2 "" V 5530 3250 50  0001 C CNN
@@
 $EndComp
 $Comp
-L C C31
+L C C1301
 U 1 1 5977530D
 P 5100 3650
-F 0 "C31" H 5125 3750 50  0000 L CNN
+F 0 "C1301" H 5125 3750 50  0000 L CNN
 F 1 "0.1uF" H 5125 3550 50  0000 L CNN
 F 2 "" H 5138 3500 50  0001 C CNN
@@
 $EndComp
 $Comp
-L C C32
+L C C1302
 U 1 1 59775333
 P 6600 3650
-F 0 "C32" H 6625 3750 50  0000 L CNN
+F 0 "C1302" H 6625 3750 50  0000 L CNN
 F 1 "0.22uF" H 6625 3550 50  0000 L CNN
 F 2 "" H 6638 3500 50  0001 C CNN
@@
 $EndComp
 $Comp
-L Earth #PWR051
+L Earth #PWR1301
 U 1 1 59775372
 P 6600 4300
-F 0 "#PWR051" H 6600 4050 50  0001 C CNN
+F 0 "#PWR1301" H 6600 4050 50  0001 C CNN
 F 1 "Earth" H 6600 4150 50  0001 C CNN
 F 2 "" H 6600 4300 50  0001 C CNN
