File: electrical/ECU/kicad_ECU/power_out_protection.sch (KiCad schematic (older format))
At the start: 16 parts, among them Q2 Q_PMOS_DGS, Q3 Q_PMOS_DGS, U9 LM2903Q2T

Commit message: minor naming change
Parts:
- renumbered 10k2 to 10k701, 10k3 to 10k702, 10k4 to 10k703, 10k5 to 10k704, C26 to C701, D4 to D701, D5 to D702, D_Zener1 to D_Zener701, Q2 to Q701, Q3 to Q702, R25 to R701, R26 to R702, R27 to R703, R28 to R704, R29 to R705, U9 to U701
Changed lines of the file:
@@
 5v_out
 $Comp
-L Q_PMOS_DGS Q2
+L Q_PMOS_DGS Q701
 U 1 1 598112D0
 P 2500 3300
-AR Path="/597003E2/598160FB/598112D0" Ref="Q2"  Part="1"
-AR Path="/5981120E/598112D0" Ref="Q5"  Part="1"
-F 0 "Q5" H 2700 3350 50  0000 L CNN
+AR Path="/597003E2/598160FB/598112D0" Ref="Q701"  Part="1"
+AR Path="/5981120E/598112D0" Ref="Q3301"  Part="1"
+F 0 "Q3301" H 2700 3350 50  0000 L CNN
 F 1 "Q_PMOS_DGS" H 2700 3250 50  0000 L CNN
 F 2 "" H 2700 3400 50  0001 C CNN
@@
 $EndComp
 $Comp
-L LM2903Q2T U9
+L LM2903Q2T U701
 U 1 1 59811370
 P 6050 4150
-AR Path="/597003E2/598160FB/59811370" Ref="U9"  Part="1"
-AR Path="/5981120E/59811370" Ref="U29"  Part="1"
-F 0 "U29" H 6050 4050 50  0000 C CNN
+AR Path="/597003E2/598160FB/59811370" Ref="U701"  Part="1"
+AR Path="/5981120E/59811370" Ref="U3301"  Part="1"
+F 0 "U3301" H 6050 4050 50  0000 C CNN
 F 1 "LM2903Q2T" H 6050 4250 50  0000 C CNN
 F 2 "MODULE" H 6050 4150 50  0001 C CNN
@@
 $EndComp
 $Comp
-L R R25
+L R R701
 U 1 1 598113F3
 P 3150 4000
-AR Path="/597003E2/598160FB/598113F3" Ref="R25"  Part="1"
-AR Path="/5981120E/598113F3" Ref="R101"  Part="1"
-F 0 "R101" V 3230 4000 50  0000 C CNN
+AR Path="/597003E2/598160FB/598113F3" Ref="R701"  Part="1"
+AR Path="/5981120E/598113F3" Ref="R3301"  Part="1"
+F 0 "R3301" V 3230 4000 50  0000 C CNN
 F 1 "300" V 3150 4000 50  0000 C CNN
 F 2 "" V 3080 4000 50  0001 C CNN
@@
 $EndComp
 $Comp
-L R 10k2
+L R 10k701
 U 1 1 5981145B
 P 2950 3600
-AR Path="/597003E2/598160FB/5981145B" Ref="10k2"  Part="1"
-AR Path="/5981120E/5981145B" Ref="10k6"  Part="1"
-F 0 "10k6" V 3030 3600 50  0000 C CNN
+AR Path="/597003E2/598160FB/5981145B" Ref="10k701"  Part="1"
+AR Path="/5981120E/5981145B" Ref="10k3301"  Part="1"
+F 0 "10k3301" V 3030 3600 50  0000 C CNN
 F 1 "10k" V 2950 3600 50  0000 C CNN
 F 2 "" V 2880 3600 50  0001 C CNN
@@
 $EndComp
 $Comp
-L D D4
+L D D701
 U 1 1 59811491
 P 3500 3600
-AR Path="/597003E2/598160FB/59811491" Ref="D4"  Part="1"
-AR Path="/5981120E/59811491" Ref="D38"  Part="1"
-F 0 "D38" H 3500 3700 50  0000 C CNN
+AR Path="/597003E2/598160FB/59811491" Ref="D701"  Part="1"
+AR Path="/5981120E/59811491" Ref="D3301"  Part="1"
+F 0 "D3301" H 3500 3700 50  0000 C CNN
 F 1 "D" H 3500 3500 50  0000 C CNN
 F 2 "" H 3500 3600 50  0001 C CNN
@@
 $EndComp
 $Comp
-L R 10k3
+L R 10k702
 U 1 1 59811538
 P 4900 3550
-AR Path="/597003E2/598160FB/59811538" Ref="10k3"  Part="1"
-AR Path="/5981120E/59811538" Ref="10k7"  Part="1"
-F 0 "10k7" V 4980 3550 50  0000 C CNN
+AR Path="/597003E2/598160FB/59811538" Ref="10k702"  Part="1"
+AR Path="/5981120E/59811538" Ref="10k3302"  Part="1"
+F 0 "10k3302" V 4980 3550 50  0000 C CNN
 F 1 "10k" V 4900 3550 50  0000 C CNN
 F 2 "" V 4830 3550 50  0001 C CNN
@@
 $EndComp
 $Comp
-L R R27
+L R R703
 U 1 1 59811580
 P 4900 4600
-AR Path="/597003E2/598160FB/59811580" Ref="R27"  Part="1"
-AR Path="/5981120E/59811580" Ref="R103"  Part="1"
-F 0 "R103" V 4980 4600 50  0000 C CNN
+AR Path="/597003E2/598160FB/59811580" Ref="R703"  Part="1"
+AR Path="/5981120E/59811580" Ref="R3303"  Part="1"
+F 0 "R3303" V 4980 4600 50  0000 C CNN
 F 1 "7.68k" V 4900 4600 50  0000 C CNN
 F 2 "" V 4830 4600 50  0001 C CNN
@@
 5v_in
 $Comp
-L R R26
+L R R702
 U 1 1 59811624
 P 4500 3600
-AR Path="/597003E2/598160FB/59811624" Ref="R26"  Part="1"
-AR Path="/5981120E/59811624" Ref="R102"  Part="1"
-F 0 "R102" V 4580 3600 50  0000 C CNN
+AR Path="/597003E2/598160FB/59811624" Ref="R702"  Part="1"
+AR Path="/5981120E/59811624" Ref="R3302"  Part="1"
+F 0 "R3302" V 4580 3600 50  0000 C CNN
 F 1 "510" V 4500 3600 50  0000 C CNN
 F 2 "" V 4430 3600 50  0001 C CNN
@@
 $EndComp
 $Comp
-L D_Zener D_Zener1
+L D_Zener D_Zener701
 U 1 1 59811697
 P 4500 4600
-AR Path="/597003E2/598160FB/59811697" Ref="D_Zener1"  Part="1"
-AR Path="/5981120E/59811697" Ref="D_Zener6"  Part="1"
-F 0 "D_Zener6" H 4500 4700 50  0000 C CNN
+AR Path="/597003E2/598160FB/59811697" Ref="D_Zener701"  Part="1"
+AR Path="/5981120E/59811697" Ref="D_Zener3301"  Part="1"
+F 0 "D_Zener3301" H 4500 4700 50  0000 C CNN
 F 1 "2.4v" H 4500 4500 50  0000 C CNN
 F 2 "" H 4500 4600 50  0001 C CNN
@@
 2.4v_REF
 $Comp
-L Earth #PWR034
+L Earth #PWR702
 U 1 1 598118C5
 P 4500 5000
-AR Path="/597003E2/598160FB/598118C5" Ref="#PWR034"  Part="1"
-AR Path="/5981120E/598118C5" Ref="#PWR083"  Part="1"
-F 0 "#PWR083" H 4500 4750 50  0001 C CNN
+AR Path="/597003E2/598160FB/598118C5" Ref="#PWR702"  Part="1"
+AR Path="/5981120E/598118C5" Ref="#PWR3302"  Part="1"
+F 0 "#PWR3302" H 4500 4750 50  0001 C CNN
 F 1 "Earth" H 4500 4850 50  0001 C CNN
 F 2 "" H 4500 5000 50  0001 C CNN
@@
 3.3v_out
 $Comp
-L Q_PMOS_DGS Q3
+L Q_PMOS_DGS Q702
 U 1 1 59811E9B
 P 9100 3400
-AR Path="/597003E2/598160FB/59811E9B" Ref="Q3"  Part="1"
-AR Path="/5981120E/59811E9B" Ref="Q6"  Part="1"
-F 0 "Q6" H 9300 3450 50  0000 L CNN
+AR Path="/597003E2/598160FB/59811E9B" Ref="Q702"  Part="1"
+AR Path="/5981120E/59811E9B" Ref="Q3302"  Part="1"
+F 0 "Q3302" H 9300 3450 50  0000 L CNN
 F 1 "Q_PMOS_DGS" H 9300 3350 50  0000 L CNN
 F 2 "" H 9300 3500 50  0001 C CNN
@@
 $EndComp
 $Comp
-L R R29
+L R R705
 U 1 1 59811EA1
 P 8450 4100
-AR Path="/597003E2/598160FB/59811EA1" Ref="R29"  Part="1"
-AR Path="/5981120E/59811EA1" Ref="R105"  Part="1"
-F 0 "R105" V 8530 4100 50  0000 C CNN
+AR Path="/597003E2/598160FB/59811EA1" Ref="R705"  Part="1"
+AR Path="/5981120E/59811EA1" Ref="R3305"  Part="1"
+F 0 "R3305" V 8530 4100 50  0000 C CNN
 F 1 "300" V 8450 4100 50  0000 C CNN
 F 2 "" V 8380 4100 50  0001 C CNN
@@
 $EndComp
 $Comp
-L R 10k5
+L R 10k704
 U 1 1 59811EA7
 P 8650 3700
-AR Path="/597003E2/598160FB/59811EA7" Ref="10k5"  Part="1"
-AR Path="/5981120E/59811EA7" Ref="10k9"  Part="1"
-F 0 "10k9" V 8730 3700 50  0000 C CNN
+AR Path="/597003E2/598160FB/59811EA7" Ref="10k704"  Part="1"
+AR Path="/5981120E/59811EA7" Ref="10k3304"  Part="1"
+F 0 "10k3304" V 8730 3700 50  0000 C CNN
 F 1 "10k" V 8650 3700 50  0000 C CNN
 F 2 "" V 8580 3700 50  0001 C CNN
@@
 $EndComp
 $Comp
-L D D5
+L D D702
 U 1 1 59811EAD
 P 8100 3700
-AR Path="/597003E2/598160FB/59811EAD" Ref="D5"  Part="1"
-AR Path="/5981120E/59811EAD" Ref="D39"  Part="1"
-F 0 "D39" H 8100 3800 50  0000 C CNN
+AR Path="/597003E2/598160FB/59811EAD" Ref="D702"  Part="1"
+AR Path="/5981120E/59811EAD" Ref="D3302"  Part="1"
+F 0 "D3302" H 8100 3800 50  0000 C CNN
 F 1 "D" H 8100 3600 50  0000 C CNN
 F 2 "" H 8100 3700 50  0001 C CNN
@@
 $EndComp
 $Comp
-L R 10k4
+L R 10k703
 U 1 1 59811EB3
 P 7750 3650
-AR Path="/597003E2/598160FB/59811EB3" Ref="10k4"  Part="1"
-AR Path="/5981120E/59811EB3" Ref="10k8"  Part="1"
-F 0 "10k8" V 7830 3650 50  0000 C CNN
+AR Path="/597003E2/598160FB/59811EB3" Ref="10k703"  Part="1"
+AR Path="/5981120E/59811EB3" Ref="10k3303"  Part="1"
+F 0 "10k3303" V 7830 3650 50  0000 C CNN
 F 1 "3.9k" V 7750 3650 50  0000 C CNN
 F 2 "" V 7680 3650 50  0001 C CNN
@@
 $EndComp
 $Comp
-L R R28
+L R R704
 U 1 1 59811EB9
 P 7750 4700
-AR Path="/597003E2/598160FB/59811EB9" Ref="R28"  Part="1"
-AR Path="/5981120E/59811EB9" Ref="R104"  Part="1"
-F 0 "R104" V 7830 4700 50  0000 C CNN
+AR Path="/597003E2/598160FB/59811EB9" Ref="R704"  Part="1"
+AR Path="/5981120E/59811EB9" Ref="R3304"  Part="1"
+F 0 "R3304" V 7830 4700 50  0000 C CNN
 F 1 "7.68k" V 7750 4700 50  0000 C CNN
 F 2 "" V 7680 4700 50  0001 C CNN
@@
 $EndComp
 $Comp
-L Earth #PWR035
+L Earth #PWR703
 U 1 1 59811EBF
 P 7750 5100
-AR Path="/597003E2/598160FB/59811EBF" Ref="#PWR035"  Part="1"
-AR Path="/5981120E/59811EBF" Ref="#PWR084"  Part="1"
-F 0 "#PWR084" H 7750 4850 50  0001 C CNN
+AR Path="/597003E2/598160FB/59811EBF" Ref="#PWR703"  Part="1"
+AR Path="/5981120E/59811EBF" Ref="#PWR3303"  Part="1"
+F 0 "#PWR3303" H 7750 4850 50  0001 C CNN
 F 1 "Earth" H 7750 4950 50  0001 C CNN
 F 2 "" H 7750 5100 50  0001 C CNN
@@
 5v_in
 $Comp
-L C C26
+L C C701
 U 1 1 599525C0
 P 2000 5650
-AR Path="/597003E2/598160FB/599525C0" Ref="C26"  Part="1"
-AR Path="/5981120E/599525C0" Ref="C75"  Part="1"
-F 0 "C75" H 2025 5750 50  0000 L CNN
+AR Path="/597003E2/598160FB/599525C0" Ref="C701"  Part="1"
+AR Path="/5981120E/599525C0" Ref="C3301"  Part="1"
+F 0 "C3301" H 2025 5750 50  0000 L CNN
 F 1 "0.1uF" H 2025 5550 50  0000 L CNN
 F 2 "" H 2038 5500 50  0001 C CNN
@@
 GND
 $Comp
-L Earth #PWR036
+L Earth #PWR701
 U 1 1 5995279B
 P 1550 6400
-AR Path="/597003E2/598160FB/5995279B" Ref="#PWR036"  Part="1"
-AR Path="/5981120E/5995279B" Ref="#PWR085"  Part="1"
-F 0 "#PWR085" H 1550 6150 50  0001 C CNN
+AR Path="/597003E2/598160FB/5995279B" Ref="#PWR701"  Part="1"
+AR Path="/5981120E/5995279B" Ref="#PWR3301"  Part="1"
+F 0 "#PWR3301" H 1550 6150 50  0001 C CNN
 F 1 "Earth" H 1550 6250 50  0001 C CNN
 F 2 "" H 1550 6400 50  0001 C CNN
