File: electrical/ECU/kicad_ECU/power_supply.sch (KiCad schematic (older format))
At the start: 17 parts, among them U3 MIC45205

Commit message: minor naming change
Parts:
- renumbered 0.1uF1 to 0.1uF201, 0.1uF2 to 0.1uF202, 0.1uF3 to 0.1uF203, 100nF1 to 100nF201, 100uF1 to 100uF201, 10k1 to 10k201, 10uF1 to 10uF201, 15pF1 to 15pF201, 220uF1 to 220uF201, 6A1 to 6A201, L1 to L201, R1 to R201, R2 to R202, R3 to R203, R4 to R204, R5 to R205, U3 to U201
Changed lines of the file:
@@
 $EndDescr
 $Comp
-L MIC45205 U3
+L MIC45205 U201
 U 1 1 597D91EA
 P 5800 3450
-F 0 "U3" H 5800 3350 50  0000 C CNN
+F 0 "U201" H 5800 3350 50  0000 C CNN
 F 1 "MIC45205" H 5800 3550 50  0000 C CNN
 F 2 "MODULE" H 5800 3450 50  0001 C CNN
@@
 NoConn ~ 6650 3200
 $Comp
-L Earth #PWR09
+L Earth #PWR206
 U 1 1 597DA944
 P 6950 3900
-F 0 "#PWR09" H 6950 3650 50  0001 C CNN
+F 0 "#PWR206" H 6950 3650 50  0001 C CNN
 F 1 "Earth" H 6950 3750 50  0001 C CNN
 F 2 "" H 6950 3900 50  0001 C CNN
@@
 $EndComp
 $Comp
-L R 10k1
+L R 10k201
 U 1 1 597DACD4
 P 4800 2500
-F 0 "10k1" V 4880 2500 50  0000 C CNN
+F 0 "10k201" V 4880 2500 50  0000 C CNN
 F 1 "R" V 4800 2500 50  0000 C CNN
 F 2 "" V 4730 2500 50  0001 C CNN
@@
 $EndComp
 $Comp
-L R R1
+L R R201
 U 1 1 597DAF82
 P 3150 3200
-F 0 "R1" V 3230 3200 50  0000 C CNN
+F 0 "R201" V 3230 3200 50  0000 C CNN
 F 1 "1.37k" V 3150 3200 50  0000 C CNN
 F 2 "" V 3080 3200 50  0001 C CNN
@@
 $EndComp
 $Comp
-L Earth #PWR010
+L Earth #PWR202
 U 1 1 597DB479
 P 3550 3900
-F 0 "#PWR010" H 3550 3650 50  0001 C CNN
+F 0 "#PWR202" H 3550 3650 50  0001 C CNN
 F 1 "Earth" H 3550 3750 50  0001 C CNN
 F 2 "" H 3550 3900 50  0001 C CNN
@@
 	4500 4200 4950 4200
 $Comp
-L C 100nF1
+L C 100nF201
 U 1 1 597DBD6A
 P 4400 4700
-F 0 "100nF1" H 4425 4800 50  0000 L CNN
+F 0 "100nF201" H 4425 4800 50  0000 L CNN
 F 1 "C" H 4425 4600 50  0000 L CNN
 F 2 "" H 4438 4550 50  0001 C CNN
@@
 $EndComp
 $Comp
-L R R2
+L R R202
 U 1 1 597DBDE5
 P 4000 4700
-F 0 "R2" V 4080 4700 50  0000 C CNN
+F 0 "R202" V 4080 4700 50  0000 C CNN
 F 1 "10k" V 4000 4700 50  0000 C CNN
 F 2 "" V 3930 4700 50  0001 C CNN
@@
 $EndComp
 $Comp
-L R R3
+L R R203
 U 1 1 597DBE14
 P 4000 5700
-F 0 "R3" V 4080 5700 50  0000 C CNN
+F 0 "R203" V 4080 5700 50  0000 C CNN
 F 1 "1.91k" V 4000 5700 50  0000 C CNN
 F 2 "" V 3930 5700 50  0001 C CNN
@@
 $EndComp
 $Comp
-L C 100uF1
+L C 100uF201
 U 1 1 597DBE45
 P 3000 4700
-F 0 "100uF1" H 3025 4800 50  0000 L CNN
+F 0 "100uF201" H 3025 4800 50  0000 L CNN
 F 1 "C" H 3025 4600 50  0000 L CNN
 F 2 "" H 3038 4550 50  0001 C CNN
@@
 Connection ~ 4400 5200
 $Comp
-L Earth #PWR011
+L Earth #PWR204
 U 1 1 597DC076
 P 4000 6300
-F 0 "#PWR011" H 4000 6050 50  0001 C CNN
+F 0 "#PWR204" H 4000 6050 50  0001 C CNN
 F 1 "Earth" H 4000 6150 50  0001 C CNN
 F 2 "" H 4000 6300 50  0001 C CNN
@@
 Connection ~ 3000 4300
 $Comp
-L C 15pF1
+L C 15pF201
 U 1 1 597DC6E9
 P 2250 3450
-F 0 "15pF1" H 2275 3550 50  0000 L CNN
+F 0 "15pF201" H 2275 3550 50  0000 L CNN
 F 1 "C" H 2275 3350 50  0000 L CNN
 F 2 "" H 2288 3300 50  0001 C CNN
@@
 Connection ~ 2250 3300
 $Comp
-L Earth #PWR012
+L Earth #PWR201
 U 1 1 597DC726
 P 2250 3750
-F 0 "#PWR012" H 2250 3500 50  0001 C CNN
+F 0 "#PWR201" H 2250 3500 50  0001 C CNN
 F 1 "Earth" H 2250 3600 50  0001 C CNN
 F 2 "" H 2250 3750 50  0001 C CNN
@@
 	2250 3600 2250 3750
 $Comp
-L Polyfuse 6A1
+L Polyfuse 6A201
 U 1 1 597DC85A
 P 3000 3400
-F 0 "6A1" V 2900 3400 50  0000 C CNN
+F 0 "6A201" V 2900 3400 50  0000 C CNN
 F 1 "Polyfuse" V 3100 3400 50  0000 C CNN
 F 2 "" H 3050 3200 50  0001 L CNN
@@
 FREQ
 $Comp
-L R R4
+L R R204
 U 1 1 597DD9AA
 P 8950 3000
-F 0 "R4" V 9030 3000 50  0000 C CNN
+F 0 "R204" V 9030 3000 50  0000 C CNN
 F 1 "100k" V 8950 3000 50  0000 C CNN
 F 2 "" V 8880 3000 50  0001 C CNN
@@
 $EndComp
 $Comp
-L R R5
+L R R205
 U 1 1 597DDA07
 P 8950 3550
-F 0 "R5" V 9030 3550 50  0000 C CNN
+F 0 "R205" V 9030 3550 50  0000 C CNN
 F 1 "1M" V 8950 3550 50  0000 C CNN
 F 2 "" V 8880 3550 50  0001 C CNN
@@
 Connection ~ 8950 3250
 $Comp
-L Earth #PWR013
+L Earth #PWR207
 U 1 1 597DDBC9
 P 8950 3900
-F 0 "#PWR013" H 8950 3650 50  0001 C CNN
+F 0 "#PWR207" H 8950 3650 50  0001 C CNN
 F 1 "Earth" H 8950 3750 50  0001 C CNN
 F 2 "" H 8950 3900 50  0001 C CNN
@@
 	8950 2850 8950 2550
 $Comp
-L C 10uF1
+L C 10uF201
 U 1 1 597DE47D
 P 3850 3700
-F 0 "10uF1" H 3875 3800 50  0000 L CNN
+F 0 "10uF201" H 3875 3800 50  0000 L CNN
 F 1 "C" H 3875 3600 50  0000 L CNN
 F 2 "" H 3888 3550 50  0001 C CNN
@@
 $EndComp
 $Comp
-L C 0.1uF3
+L C 0.1uF203
 U 1 1 597DE4AC
 P 4150 3700
-F 0 "0.1uF3" H 4175 3800 50  0000 L CNN
+F 0 "0.1uF203" H 4175 3800 50  0000 L CNN
 F 1 "C" H 4175 3600 50  0000 L CNN
 F 2 "" H 4188 3550 50  0001 C CNN
@@
 $EndComp
 $Comp
-L Earth #PWR014
+L Earth #PWR203
 U 1 1 597DE509
 P 3850 3900
-F 0 "#PWR014" H 3850 3650 50  0001 C CNN
+F 0 "#PWR203" H 3850 3650 50  0001 C CNN
 F 1 "Earth" H 3850 3750 50  0001 C CNN
 F 2 "" H 3850 3900 50  0001 C CNN
@@
 	3850 3850 3850 3900
 $Comp
-L Earth #PWR015
+L Earth #PWR205
 U 1 1 597DE53C
 P 4150 3900
-F 0 "#PWR015" H 4150 3650 50  0001 C CNN
+F 0 "#PWR205" H 4150 3650 50  0001 C CNN
 F 1 "Earth" H 4150 3750 50  0001 C CNN
 F 2 "" H 4150 3900 50  0001 C CNN
@@
 Connection ~ 4150 3400
 $Comp
-L C 0.1uF1
+L C 0.1uF201
 U 1 1 597DE7F9
 P 3300 4700
-F 0 "0.1uF1" H 3325 4800 50  0000 L CNN
+F 0 "0.1uF201" H 3325 4800 50  0000 L CNN
 F 1 "C" H 3325 4600 50  0000 L CNN
 F 2 "" H 3338 4550 50  0001 C CNN
@@
 $EndComp
 $Comp
-L C 0.1uF2
+L C 0.1uF202
 U 1 1 597DE82E
 P 3600 4700
-F 0 "0.1uF2" H 3625 4800 50  0000 L CNN
+F 0 "0.1uF202" H 3625 4800 50  0000 L CNN
 F 1 "C" H 3625 4600 50  0000 L CNN
 F 2 "" H 3638 4550 50  0001 C CNN
@@
 Connection ~ 3300 5150
 $Comp
-L CP1 220uF1
+L CP1 220uF201
 U 1 1 597DEB54
 P 3550 3700
-F 0 "220uF1" H 3575 3800 50  0000 L CNN
+F 0 "220uF201" H 3575 3800 50  0000 L CNN
 F 1 "CP1" H 3575 3600 50  0000 L CNN
 F 2 "" H 3550 3700 50  0001 C CNN
@@
 $EndComp
 $Comp
-L Ferrite_Bead L1
+L Ferrite_Bead L201
 U 1 1 5980C8ED
 P 2300 4300
-F 0 "L1" V 2150 4325 50  0000 C CNN
+F 0 "L201" V 2150 4325 50  0000 C CNN
 F 1 "Ferrite_Bead" V 2450 4300 50  0000 C CNN
 F 2 "" V 2230 4300 50  0001 C CNN
@@
 Connection ~ 6800 3400
 $Comp
-L PWR_FLAG #FLG016
+L PWR_FLAG #FLG201
 U 1 1 597DDEFE
 P 2700 4300
-F 0 "#FLG016" H 2700 4375 50  0001 C CNN
+F 0 "#FLG201" H 2700 4375 50  0001 C CNN
 F 1 "PWR_FLAG" H 2700 4450 50  0000 C CNN
 F 2 "" H 2700 4300 50  0001 C CNN
@@
 $EndComp
 $Comp
-L PWR_FLAG #FLG017
+L PWR_FLAG #FLG202
 U 1 1 59964D54
 P 3250 3400
-F 0 "#FLG017" H 3250 3495 50  0001 C CNN
+F 0 "#FLG202" H 3250 3495 50  0001 C CNN
 F 1 "PWR_FLAG" H 3250 3580 50  0000 C CNN
 F 2 "" H 3250 3400 50  0000 C CNN
