File: electrical/ECU/kicad_ECU/usb.sch (KiCad schematic (older format))
At the start: 23 parts, among them J1 USB_OTG, Q1 2N7002, U6 USBULC6-2M6, U7 FT231XQ

Commit message: minor naming change
Parts:
- renumbered C14 to C501, C15 to C502, C16 to C503, C17 to C504, C18 to C505, C19 to C506, C20 to C507, C21 to C508, D2 to D501, D3 to D502, F1 to F501, J1 to J501, L3 to L501, L4 to L502, Q1 to Q501, R17 to R501, R18 to R502, R19 to R503, R20 to R504, R21 to R505, R22 to R506, U6 to U501, U7 to U502
Changed lines of the file:
@@
 $EndDescr
 $Comp
-L FT231XQ U7
+L FT231XQ U502
 U 1 1 5970A7F7
 P 5800 3850
-F 0 "U7" H 5250 4650 50  0000 L CNN
+F 0 "U502" H 5250 4650 50  0000 L CNN
 F 1 "FT231XQ" H 6050 4650 50  0000 L CNN
 F 2 "QFN-20" H 5800 3850 50  0001 C CNN
@@
 $EndComp
 $Comp
-L USB_OTG-RESCUE-airhead_ecu J1
+L USB_OTG-RESCUE-airhead_ecu J501
 U 1 1 5970A804
 P 1650 3550
-F 0 "J1" H 1450 4000 50  0000 L CNN
+F 0 "J501" H 1450 4000 50  0000 L CNN
 F 1 "USB_OTG" H 1450 3900 50  0000 L CNN
 F 2 "" H 1800 3500 50  0001 C CNN
@@
 $EndComp
 $Comp
-L C C15
+L C C502
 U 1 1 5970A811
 P 4050 4500
-F 0 "C15" H 4075 4600 50  0000 L CNN
+F 0 "C502" H 4075 4600 50  0000 L CNN
 F 1 "47pF" H 4075 4400 50  0000 L CNN
 F 2 "" H 4088 4350 50  0001 C CNN
@@
 $EndComp
 $Comp
-L C C16
+L C C503
 U 1 1 5970A818
 P 4300 4500
-F 0 "C16" H 4325 4600 50  0000 L CNN
+F 0 "C503" H 4325 4600 50  0000 L CNN
 F 1 "47pF" H 4325 4400 50  0000 L CNN
 F 2 "" H 4338 4350 50  0001 C CNN
@@
 $EndComp
 $Comp
-L R R17
+L R R501
 U 1 1 5970A81F
 P 4550 3550
-F 0 "R17" V 4630 3550 50  0000 C CNN
+F 0 "R501" V 4630 3550 50  0000 C CNN
 F 1 "27R" V 4550 3550 50  0000 C CNN
 F 2 "" V 4480 3550 50  0001 C CNN
@@
 $EndComp
 $Comp
-L R R18
+L R R502
 U 1 1 5970A826
 P 4750 3650
-F 0 "R18" V 4830 3650 50  0000 C CNN
+F 0 "R502" V 4830 3650 50  0000 C CNN
 F 1 "27R" V 4750 3650 50  0000 C CNN
 F 2 "" V 4680 3650 50  0001 C CNN
@@
 $EndComp
 $Comp
-L Ferrite_Bead L4
+L Ferrite_Bead L502
 U 1 1 5970A82D
 P 4050 2700
-F 0 "L4" V 3900 2725 50  0000 C CNN
+F 0 "L502" V 3900 2725 50  0000 C CNN
 F 1 "Ferrite_Bead" V 4200 2700 50  0000 C CNN
 F 2 "" V 3980 2700 50  0001 C CNN
@@
 $EndComp
 $Comp
-L C C19
+L C C506
 U 1 1 5970A834
 P 4950 4500
-F 0 "C19" H 4975 4600 50  0000 L CNN
+F 0 "C506" H 4975 4600 50  0000 L CNN
 F 1 "100nF" H 4975 4400 50  0000 L CNN
 F 2 "" H 4988 4350 50  0001 C CNN
@@
 $EndComp
 $Comp
-L C C17
+L C C504
 U 1 1 5970A868
 P 4400 2850
-F 0 "C17" H 4425 2950 50  0000 L CNN
+F 0 "C504" H 4425 2950 50  0000 L CNN
 F 1 "100nF" H 4425 2750 50  0000 L CNN
 F 2 "" H 4438 2700 50  0001 C CNN
@@
 $EndComp
 $Comp
-L C C18
+L C C505
 U 1 1 5970A86F
 P 4700 2850
-F 0 "C18" H 4725 2950 50  0000 L CNN
+F 0 "C505" H 4725 2950 50  0000 L CNN
 F 1 "4.7uF" H 4725 2750 50  0000 L CNN
 F 2 "" H 4738 2700 50  0001 C CNN
@@
 $EndComp
 $Comp
-L Earth #PWR027
+L Earth #PWR502
 U 1 1 5970A87F
 P 4700 3100
-F 0 "#PWR027" H 4700 2850 50  0001 C CNN
+F 0 "#PWR502" H 4700 2850 50  0001 C CNN
 F 1 "Earth" H 4700 2950 50  0001 C CNN
 F 2 "" H 4700 3100 50  0001 C CNN
@@
 $EndComp
 $Comp
-L C C14
+L C C501
 U 1 1 5970A887
 P 3800 4500
-F 0 "C14" H 3825 4600 50  0000 L CNN
+F 0 "C501" H 3825 4600 50  0000 L CNN
 F 1 "10nF" H 3825 4400 50  0000 L CNN
 F 2 "" H 3838 4350 50  0001 C CNN
@@
 5VDC
 $Comp
-L PWR_FLAG #FLG028
+L PWR_FLAG #FLG502
 U 1 1 5970A92F
 P 3800 2400
-F 0 "#FLG028" H 3800 2475 50  0001 C CNN
+F 0 "#FLG502" H 3800 2475 50  0001 C CNN
 F 1 "PWR_FLAG" H 3800 2550 50  0000 C CNN
 F 2 "" H 3800 2400 50  0001 C CNN
@@
 $EndComp
 $Comp
-L LED-RESCUE-airhead_ecu D2
+L LED-RESCUE-airhead_ecu D501
 U 1 1 5970AB1A
 P 7400 3750
-F 0 "D2" H 7400 3850 50  0000 C CNN
+F 0 "D501" H 7400 3850 50  0000 C CNN
 F 1 "RED" H 7400 3650 50  0000 C CNN
 F 2 "" H 7400 3750 50  0001 C CNN
@@
 $EndComp
 $Comp
-L LED-RESCUE-airhead_ecu D3
+L LED-RESCUE-airhead_ecu D502
 U 1 1 5970AB4D
 P 7800 3750
-F 0 "D3" H 7800 3850 50  0000 C CNN
+F 0 "D502" H 7800 3850 50  0000 C CNN
 F 1 "YELLOW" H 7800 3650 50  0000 C CNN
 F 2 "" H 7800 3750 50  0001 C CNN
@@
 $EndComp
 $Comp
-L R R19
+L R R503
 U 1 1 5970AB82
 P 7400 3150
-F 0 "R19" V 7480 3150 50  0000 C CNN
+F 0 "R503" V 7480 3150 50  0000 C CNN
 F 1 "270R" V 7400 3150 50  0000 C CNN
 F 2 "" V 7330 3150 50  0001 C CNN
@@
 $EndComp
 $Comp
-L R R20
+L R R504
 U 1 1 5970ABB3
 P 7800 3150
-F 0 "R20" V 7880 3150 50  0000 C CNN
+F 0 "R504" V 7880 3150 50  0000 C CNN
 F 1 "270R" V 7800 3150 50  0000 C CNN
 F 2 "" V 7730 3150 50  0001 C CNN
@@
 3.3VDC
 $Comp
-L 2N7002 Q1
+L 2N7002 Q501
 U 1 1 5970B61B
 P 9700 2050
-F 0 "Q1" H 9900 2125 50  0000 L CNN
+F 0 "Q501" H 9900 2125 50  0000 L CNN
 F 1 "2N7002" H 9900 2050 50  0000 L CNN
 F 2 "TO_SOT_Packages_SMD:SOT-23" H 9900 1975 50  0001 L CIN
@@
 RESET
 $Comp
-L R R22
+L R R506
 U 1 1 5970B767
 P 10100 1800
-F 0 "R22" V 10180 1800 50  0000 C CNN
+F 0 "R506" V 10180 1800 50  0000 C CNN
 F 1 "10k" V 10100 1800 50  0000 C CNN
 F 2 "" V 10030 1800 50  0001 C CNN
@@
 3.3VDC
 $Comp
-L R R21
+L R R505
 U 1 1 5970BC14
 P 9300 1800
-F 0 "R21" V 9380 1800 50  0000 C CNN
+F 0 "R505" V 9380 1800 50  0000 C CNN
 F 1 "10K" V 9300 1800 50  0000 C CNN
 F 2 "" V 9230 1800 50  0001 C CNN
@@
 5VDC
 $Comp
-L C C21
+L C C508
 U 1 1 5970C0C1
 P 7100 5900
-F 0 "C21" H 7125 6000 50  0000 L CNN
+F 0 "C508" H 7125 6000 50  0000 L CNN
 F 1 "0.1uF" H 7125 5800 50  0000 L CNN
 F 2 "" H 7138 5750 50  0001 C CNN
@@
 $EndComp
 $Comp
-L CP1 C20
+L CP1 C507
 U 1 1 5970C14D
 P 7100 5250
-F 0 "C20" H 7125 5350 50  0000 L CNN
+F 0 "C507" H 7125 5350 50  0000 L CNN
 F 1 "10uF" H 7125 5150 50  0000 L CNN
 F 2 "" H 7100 5250 50  0001 C CNN
@@
 $EndComp
 $Comp
-L PTC_FUSE F1
+L PTC_FUSE F501
 U 1 1 597385D0
 P 3450 3350
-F 0 "F1" H 3450 3250 60  0000 C CNN
+F 0 "F501" H 3450 3250 60  0000 C CNN
 F 1 "500mA" H 3450 3150 60  0000 C CNN
 F 2 "" H 3450 3350 60  0000 C CNN
@@
 $EndComp
 $Comp
-L USBULC6-2M6 U6
+L USBULC6-2M6 U501
 U 1 1 5973E25B
 P 2750 4000
-F 0 "U6" H 2750 4225 39  0000 C CNN
+F 0 "U501" H 2750 4225 39  0000 C CNN
 F 1 "USBULC6-2M6" H 2750 3775 39  0000 C CNN
 F 2 "" H 2225 4950 39  0000 C CNN
@@
 $EndComp
 $Comp
-L Ferrite_Bead L3
+L Ferrite_Bead L501
 U 1 1 5973EA8C
 P 2750 4950
-F 0 "L3" V 2600 4975 50  0000 C CNN
+F 0 "L501" V 2600 4975 50  0000 C CNN
 F 1 "Ferrite_Bead" V 2900 4950 50  0000 C CNN
 F 2 "" V 2680 4950 50  0001 C CNN
@@
 $EndComp
 $Comp
-L Earth #PWR029
+L Earth #PWR501
 U 1 1 5973EE3A
 P 1650 6050
-F 0 "#PWR029" H 1650 5800 50  0001 C CNN
+F 0 "#PWR501" H 1650 5800 50  0001 C CNN
 F 1 "Earth" H 1650 5900 50  0001 C CNN
 F 2 "" H 1650 6050 50  0001 C CNN
@@
 Connection ~ 6750 5250
 $Comp
-L PWR_FLAG #FLG030
+L PWR_FLAG #FLG501
 U 1 1 599185CD
 P 2300 3350
-F 0 "#FLG030" H 2300 3425 50  0001 C CNN
+F 0 "#FLG501" H 2300 3425 50  0001 C CNN
 F 1 "PWR_FLAG" H 2300 3500 50  0000 C CNN
 F 2 "" H 2300 3350 50  0001 C CNN
@@
 Connection ~ 3800 2700
 $Comp
-L PWR_FLAG #FLG031
+L PWR_FLAG #FLG503
 U 1 1 59918807
 P 4600 2300
-F 0 "#FLG031" H 4600 2375 50  0001 C CNN
+F 0 "#FLG503" H 4600 2375 50  0001 C CNN
 F 1 "PWR_FLAG" H 4600 2450 50  0000 C CNN
 F 2 "" H 4600 2300 50  0001 C CNN
