File: electrical/ECU/kicad_ECU/vin_reg.sch (KiCad schematic (older format))
At the start: 10 parts, among them Q4 Q_PMOS_DGS, U10 MC78M05CDT

Commit message: minor naming change
Parts:
- renumbered 30V1A1 to 30V1A1001, C27 to C1001, C28 to C1002, C29 to C1003, C30 to C1004, Q4 to Q1001, R30 to R1001, R31 to R1002, U10 to U1001, ZENER1 to ZENER1001
Changed lines of the file:
@@
 5v
 $Comp
-L ZENER 30V1A1
+L ZENER 30V1A1001
 U 1 1 598E15FE
 P 4050 2550
-F 0 "30V1A1" H 4050 2650 50  0000 C CNN
+F 0 "30V1A1001" H 4050 2650 50  0000 C CNN
 F 1 "ZENER" H 4050 2450 50  0000 C CNN
 F 2 "" H 4050 2550 50  0000 C CNN
@@
 $EndComp
 $Comp
-L MC78M05CDT U10
+L MC78M05CDT U1001
 U 1 1 598E1622
 P 5500 2600
-F 0 "U10" H 5300 2800 50  0000 C CNN
+F 0 "U1001" H 5300 2800 50  0000 C CNN
 F 1 "MC78M05CDT" H 5500 2800 50  0000 L CNN
 F 2 "TO-252" H 5500 2700 50  0000 C CIN
@@
 $EndComp
 $Comp
-L C C27
+L C C1001
 U 1 1 598E1651
 P 4650 2900
-F 0 "C27" H 4675 3000 50  0000 L CNN
+F 0 "C1001" H 4675 3000 50  0000 L CNN
 F 1 "0.1uF" H 4675 2800 50  0000 L CNN
 F 2 "" H 4688 2750 50  0000 C CNN
@@
 $EndComp
 $Comp
-L C C29
+L C C1003
 U 1 1 598E1685
 P 6900 2900
-F 0 "C29" H 6925 3000 50  0000 L CNN
+F 0 "C1003" H 6925 3000 50  0000 L CNN
 F 1 "10uF" H 6925 2800 50  0000 L CNN
 F 2 "" H 6938 2750 50  0000 C CNN
@@
 $EndComp
 $Comp
-L C C30
+L C C1004
 U 1 1 598E16FC
 P 7400 2900
-F 0 "C30" H 7425 3000 50  0000 L CNN
+F 0 "C1004" H 7425 3000 50  0000 L CNN
 F 1 "0.1uF" H 7425 2800 50  0000 L CNN
 F 2 "" H 7438 2750 50  0000 C CNN
@@
 $EndComp
 $Comp
-L Q_PMOS_DGS Q4
+L Q_PMOS_DGS Q1001
 U 1 1 598E1750
 P 5500 4200
-F 0 "Q4" H 5800 4250 50  0000 R CNN
+F 0 "Q1001" H 5800 4250 50  0000 R CNN
 F 1 "Q_PMOS_DGS" H 6150 4150 50  0000 R CNN
 F 2 "" H 5700 4300 50  0000 C CNN
@@
 $EndComp
 $Comp
-L ZENER ZENER1
+L ZENER ZENER1001
 U 1 1 598E17AF
 P 5500 5150
-F 0 "ZENER1" H 5500 5250 50  0000 C CNN
+F 0 "ZENER1001" H 5500 5250 50  0000 C CNN
 F 1 "5.1V" H 5500 5050 50  0000 C CNN
 F 2 "" H 5500 5150 50  0000 C CNN
@@
 $EndComp
 $Comp
-L R R31
+L R R1002
 U 1 1 598E17EF
 P 4800 5100
-F 0 "R31" V 4880 5100 50  0000 C CNN
+F 0 "R1002" V 4880 5100 50  0000 C CNN
 F 1 "100k" V 4800 5100 50  0000 C CNN
 F 2 "" V 4730 5100 50  0000 C CNN
@@
 $EndComp
 $Comp
-L R R30
+L R R1001
 U 1 1 598E182B
 P 4200 4800
-F 0 "R30" V 4280 4800 50  0000 C CNN
+F 0 "R1001" V 4280 4800 50  0000 C CNN
 F 1 "3.9k" V 4200 4800 50  0000 C CNN
 F 2 "" V 4130 4800 50  0000 C CNN
@@
 $EndComp
 $Comp
-L C C28
+L C C1002
 U 1 1 598E186D
 P 6400 5050
-F 0 "C28" H 6425 5150 50  0000 L CNN
+F 0 "C1002" H 6425 5150 50  0000 L CNN
 F 1 "10uF" H 6425 4950 50  0000 L CNN
 F 2 "" H 6438 4900 50  0000 C CNN
@@
 Connection ~ 4800 4800
 $Comp
-L Earth #PWR043
+L Earth #PWR1001
 U 1 1 598E1983
 P 4650 3200
-F 0 "#PWR043" H 4650 2950 50  0001 C CNN
+F 0 "#PWR1001" H 4650 2950 50  0001 C CNN
 F 1 "Earth" H 4650 3050 50  0001 C CNN
 F 2 "" H 4650 3200 50  0000 C CNN
@@
 $EndComp
 $Comp
-L Earth #PWR044
+L Earth #PWR1003
 U 1 1 598E19AB
 P 5500 3200
-F 0 "#PWR044" H 5500 2950 50  0001 C CNN
+F 0 "#PWR1003" H 5500 2950 50  0001 C CNN
 F 1 "Earth" H 5500 3050 50  0001 C CNN
 F 2 "" H 5500 3200 50  0000 C CNN
@@
 $EndComp
 $Comp
-L Earth #PWR045
+L Earth #PWR1006
 U 1 1 598E19D3
 P 6900 3200
-F 0 "#PWR045" H 6900 2950 50  0001 C CNN
+F 0 "#PWR1006" H 6900 2950 50  0001 C CNN
 F 1 "Earth" H 6900 3050 50  0001 C CNN
 F 2 "" H 6900 3200 50  0000 C CNN
@@
 $EndComp
 $Comp
-L Earth #PWR046
+L Earth #PWR1007
 U 1 1 598E19FB
 P 7400 3200
-F 0 "#PWR046" H 7400 2950 50  0001 C CNN
+F 0 "#PWR1007" H 7400 2950 50  0001 C CNN
 F 1 "Earth" H 7400 3050 50  0001 C CNN
 F 2 "" H 7400 3200 50  0000 C CNN
@@
 $EndComp
 $Comp
-L Earth #PWR047
+L Earth #PWR1002
 U 1 1 598E1A23
 P 4800 5550
-F 0 "#PWR047" H 4800 5300 50  0001 C CNN
+F 0 "#PWR1002" H 4800 5300 50  0001 C CNN
 F 1 "Earth" H 4800 5400 50  0001 C CNN
 F 2 "" H 4800 5550 50  0000 C CNN
@@
 $EndComp
 $Comp
-L Earth #PWR048
+L Earth #PWR1004
 U 1 1 598E1A4B
 P 5500 5550
-F 0 "#PWR048" H 5500 5300 50  0001 C CNN
+F 0 "#PWR1004" H 5500 5300 50  0001 C CNN
 F 1 "Earth" H 5500 5400 50  0001 C CNN
 F 2 "" H 5500 5550 50  0000 C CNN
@@
 $EndComp
 $Comp
-L Earth #PWR049
+L Earth #PWR1005
 U 1 1 598E1A73
 P 6400 5550
-F 0 "#PWR049" H 6400 5300 50  0001 C CNN
+F 0 "#PWR1005" H 6400 5300 50  0001 C CNN
 F 1 "Earth" H 6400 5400 50  0001 C CNN
 F 2 "" H 6400 5550 50  0000 C CNN
