File: electrical/ECU/kicad_ECU/vr.sch (KiCad schematic (older format))
At the start: 2 parts, among them U4 L9484

Commit message: minor naming change
Parts:
- renumbered TH1 to TH301, U4 to U301
Changed lines of the file:
@@
 $EndDescr
 $Comp
-L L9484 U4
+L L9484 U301
 U 1 1 58AD6AAA
 P 6800 3700
-F 0 "U4" H 6850 3750 50  0000 C CNN
+F 0 "U301" H 6850 3750 50  0000 C CNN
 F 1 "L9484" H 6800 3800 50  0000 C CNN
 F 2 "MODULE" H 6800 3700 50  0001 C CNN
@@
 $EndComp
 $Comp
-L Thermistor_NTC TH1
+L Thermistor_NTC TH301
 U 1 1 58AD6AB1
 P 5300 3500
-F 0 "TH1" V 5125 3500 50  0000 C CNN
+F 0 "TH301" V 5125 3500 50  0000 C CNN
 F 1 "Thermistor_NTC" V 5425 3500 50  0000 C CNN
 F 2 "" H 5300 3550 50  0001 C CNN
@@
 Connection ~ 5750 3750
 $Comp
-L Earth #PWR018
+L Earth #PWR301
 U 1 1 58AD6ACC
 P 5500 4450
-F 0 "#PWR018" H 5500 4200 50  0001 C CNN
+F 0 "#PWR301" H 5500 4200 50  0001 C CNN
 F 1 "Earth" H 5500 4300 50  0001 C CNN
 F 2 "" H 5500 4450 50  0000 C CNN
